File: hardware/stm32-wifi-door-bell-input.sch (KiCad schematic (older format))
At the start: 24 parts, among them P4 P02, P5 P03, U5 OPAMP-DUAL, U7 OPAMP-DUAL, U8 OPAMP-DUAL, U9 OPAMP-DUAL

Commit message: more schematic work
Parts:
- P4: value P02 -> FRONT
- P5: value P03 -> BACK
Changed lines of the file:
@@
 $Descr A4 11693 8268
 encoding utf-8
-Sheet 2 3
+Sheet 2 6
 Title ""
 Date ""
@@
 P 1300 1900
 F 0 "P4" H 1350 1950 60  0000 C CNN
-F 1 "P02" H 1300 1550 60  0000 L CNN
+F 1 "FRONT" H 1300 1550 60  0000 L CNN
 F 2 "" H 1300 1900 60  0000 C CNN
 F 3 "" H 1300 1900 60  0000 C CNN
@@
 $EndComp
 $Comp
-L GNDPWR #PWR026
+L GNDPWR #PWR17
 U 1 1 54B1A9EE
 P 1700 2400
-F 0 "#PWR026" H 1700 2450 40  0001 C CNN
+F 0 "#PWR17" H 1700 2450 40  0001 C CNN
 F 1 "GNDPWR" H 1700 2320 40  0001 C CNN
 F 2 "" H 1700 2400 60  0000 C CNN
@@
 $EndComp
 $Comp
-L GNDPWR #PWR027
+L GNDPWR #PWR22
 U 1 1 54B1AA1B
 P 3200 2600
-F 0 "#PWR027" H 3200 2650 40  0001 C CNN
+F 0 "#PWR22" H 3200 2650 40  0001 C CNN
 F 1 "GNDPWR" H 3200 2520 40  0001 C CNN
 F 2 "" H 3200 2600 60  0000 C CNN
@@
 	2400 2000 2300 2000
 $Comp
-L Vcc #PWR028
+L Vcc #PWR21
 U 1 1 54B1AA25
 P 3200 1400
-F 0 "#PWR028" H 3200 1490 20  0001 C CNN
+F 0 "#PWR21" H 3200 1490 20  0001 C CNN
 F 1 "Vcc" H 3200 1490 30  0000 C CNN
 F 2 "" H 3200 1400 60  0000 C CNN
@@
 	2700 1800 2700 2600
 $Comp
-L GNDPWR #PWR029
+L GNDPWR #PWR19
 U 1 1 54B1AA33
 P 2700 2600
-F 0 "#PWR029" H 2700 2650 40  0001 C CNN
+F 0 "#PWR19" H 2700 2650 40  0001 C CNN
 F 1 "GNDPWR" H 2700 2520 40  0001 C CNN
 F 2 "" H 2700 2600 60  0000 C CNN
@@
 Connection ~ 4100 2100
 $Comp
-L GNDPWR #PWR030
+L GNDPWR #PWR26
 U 1 1 54B1AA4B
 P 4100 2600
-F 0 "#PWR030" H 4100 2650 40  0001 C CNN
+F 0 "#PWR26" H 4100 2650 40  0001 C CNN
 F 1 "GNDPWR" H 4100 2520 40  0001 C CNN
 F 2 "" H 4100 2600 60  0000 C CNN
@@
 	4100 2400 4100 2600
 $Comp
-L Vcc #PWR031
+L Vcc #PWR25
 U 1 1 54B1AA52
 P 4100 1400
-F 0 "#PWR031" H 4100 1490 20  0001 C CNN
+F 0 "#PWR25" H 4100 1490 20  0001 C CNN
 F 1 "Vcc" H 4100 1490 30  0000 C CNN
 F 2 "" H 4100 1400 60  0000 C CNN
@@
 P 1300 4200
 F 0 "P5" H 1350 4250 60  0000 C CNN
-F 1 "P03" H 1300 3850 60  0000 L CNN
+F 1 "BACK" H 1300 3850 60  0000 L CNN
 F 2 "" H 1300 4200 60  0000 C CNN
 F 3 "" H 1300 4200 60  0000 C CNN
@@
 $EndComp
 $Comp
-L GNDPWR #PWR032
+L GNDPWR #PWR18
 U 1 1 54B1F484
 P 1700 4700
-F 0 "#PWR032" H 1700 4750 40  0001 C CNN
+F 0 "#PWR18" H 1700 4750 40  0001 C CNN
 F 1 "GNDPWR" H 1700 4620 40  0001 C CNN
 F 2 "" H 1700 4700 60  0000 C CNN
@@
 $EndComp
 $Comp
-L GNDPWR #PWR033
+L GNDPWR #PWR29
 U 1 1 54B1FBB7
 P 5400 2600
-F 0 "#PWR033" H 5400 2650 40  0001 C CNN
+F 0 "#PWR29" H 5400 2650 40  0001 C CNN
 F 1 "GNDPWR" H 5400 2520 40  0001 C CNN
 F 2 "" H 5400 2600 60  0000 C CNN
@@
 Connection ~ 5700 2200
 $Comp
-L GNDPWR #PWR034
+L GNDPWR #PWR32
 U 1 1 54B1FF14
 P 5700 2600
-F 0 "#PWR034" H 5700 2650 40  0001 C CNN
+F 0 "#PWR32" H 5700 2650 40  0001 C CNN
 F 1 "GNDPWR" H 5700 2520 40  0001 C CNN
 F 2 "" H 5700 2600 60  0000 C CNN
@@
 	5700 2500 5700 2600
 $Comp
-L Vcc #PWR035
+L Vcc #PWR31
 U 1 1 54B1FF62
 P 5700 1400
-F 0 "#PWR035" H 5700 1490 20  0001 C CNN
+F 0 "#PWR31" H 5700 1490 20  0001 C CNN
 F 1 "Vcc" H 5700 1490 30  0000 C CNN
 F 2 "" H 5700 1400 60  0000 C CNN
@@
 	5700 1400 5700 1700
 $Comp
-L GNDPWR #PWR036
+L GNDPWR #PWR36
 U 1 1 54B20160
 P 6200 2600
-F 0 "#PWR036" H 6200 2650 40  0001 C CNN
+F 0 "#PWR36" H 6200 2650 40  0001 C CNN
 F 1 "GNDPWR" H 6200 2520 40  0001 C CNN
 F 2 "" H 6200 2600 60  0000 C CNN
@@
 	6200 2400 6200 2600
 $Comp
-L +3.3V #PWR037
+L +3.3V #PWR35
 U 1 1 54B201A4
 P 6200 1400
-F 0 "#PWR037" H 6200 1490 20  0001 C CNN
+F 0 "#PWR35" H 6200 1490 20  0001 C CNN
 F 1 "+3.3V" H 6200 1490 30  0000 C CNN
 F 2 "" H 6200 1400 60  0000 C CNN
@@
 $EndComp
 $Comp
-L GNDPWR #PWR038
+L GNDPWR #PWR24
 U 1 1 54B20FC2
 P 3200 4900
-F 0 "#PWR038" H 3200 4950 40  0001 C CNN
+F 0 "#PWR24" H 3200 4950 40  0001 C CNN
 F 1 "GNDPWR" H 3200 4820 40  0001 C CNN
 F 2 "" H 3200 4900 60  0000 C CNN
@@
 Connection ~ 2800 4300
 $Comp
-L Vcc #PWR039
+L Vcc #PWR23
 U 1 1 54B20FCB
 P 3200 3700
-F 0 "#PWR039" H 3200 3790 20  0001 C CNN
+F 0 "#PWR23" H 3200 3790 20  0001 C CNN
 F 1 "Vcc" H 3200 3790 30  0000 C CNN
 F 2 "" H 3200 3700 60  0000 C CNN
@@
 	2700 4100 2700 4900
 $Comp
-L GNDPWR #PWR040
+L GNDPWR #PWR20
 U 1 1 54B20FD9
 P 2700 4900
-F 0 "#PWR040" H 2700 4950 40  0001 C CNN
+F 0 "#PWR20" H 2700 4950 40  0001 C CNN
 F 1 "GNDPWR" H 2700 4820 40  0001 C CNN
 F 2 "" H 2700 4900 60  0000 C CNN
@@
 Connection ~ 4100 4400
 $Comp
-L GNDPWR #PWR041
+L GNDPWR #PWR28
 U 1 1 54B20FEF
 P 4100 4900
-F 0 "#PWR041" H 4100 4950 40  0001 C CNN
+F 0 "#PWR28" H 4100 4950 40  0001 C CNN
 F 1 "GNDPWR" H 4100 4820 40  0001 C CNN
 F 2 "" H 4100 4900 60  0000 C CNN
@@
 	4100 4700 4100 4900
 $Comp
-L Vcc #PWR042
+L Vcc #PWR27
 U 1 1 54B20FF6
 P 4100 3700
-F 0 "#PWR042" H 4100 3790 20  0001 C CNN
+F 0 "#PWR27" H 4100 3790 20  0001 C CNN
 F 1 "Vcc" H 4100 3790 30  0000 C CNN
 F 2 "" H 4100 3700 60  0000 C CNN
@@
 $EndComp
 $Comp
-L GNDPWR #PWR043
+L GNDPWR #PWR30
 U 1 1 54B21009
 P 5400 4900
-F 0 "#PWR043" H 5400 4950 40  0001 C CNN
+F 0 "#PWR30" H 5400 4950 40  0001 C CNN
 F 1 "GNDPWR" H 5400 4820 40  0001 C CNN
 F 2 "" H 5400 4900 60  0000 C CNN
@@
 Connection ~ 5700 4500
 $Comp
-L GNDPWR #PWR044
+L GNDPWR #PWR34
 U 1 1 54B21029
 P 5700 4900
-F 0 "#PWR044" H 5700 4950 40  0001 C CNN
+F 0 "#PWR34" H 5700 4950 40  0001 C CNN
 F 1 "GNDPWR" H 5700 4820 40  0001 C CNN
 F 2 "" H 5700 4900 60  0000 C CNN
@@
 	5700 4800 5700 4900
 $Comp
-L Vcc #PWR045
+L Vcc #PWR33
 U 1 1 54B21030
 P 5700 3700
-F 0 "#PWR045" H 5700 3790 20  0001 C CNN
+F 0 "#PWR33" H 5700 3790 20  0001 C CNN
 F 1 "Vcc" H 5700 3790 30  0000 C CNN
 F 2 "" H 5700 3700 60  0000 C CNN
@@
 	5700 3700 5700 4000
 $Comp
-L GNDPWR #PWR046
+L GNDPWR #PWR38
 U 1 1 54B21037
 P 6200 4900
-F 0 "#PWR046" H 6200 4950 40  0001 C CNN
+F 0 "#PWR38" H 6200 4950 40  0001 C CNN
 F 1 "GNDPWR" H 6200 4820 40  0001 C CNN
 F 2 "" H 6200 4900 60  0000 C CNN
@@
 	6200 4700 6200 4900
 $Comp
-L +3.3V #PWR047
+L +3.3V #PWR37
 U 1 1 54B2103E
 P 6200 3700
-F 0 "#PWR047" H 6200 3790 20  0001 C CNN
+F 0 "#PWR37" H 6200 3790 20  0001 C CNN
 F 1 "+3.3V" H 6200 3790 30  0000 C CNN
 F 2 "" H 6200 3700 60  0000 C CNN

Commit message: reannotate schematic
Parts:
- removed unit 2 of U7
- removed unit 2 of U9
- renumbered D3 to D201, D6 to D202, P4 to P201, P5 to P202, R10 to R201, R21 to R202, R11 to R203, R22 to R204, R12 to R205, R13 to R206, R23 to R207, R24 to R208, R17 to R209, R25 to R210, R18 to R211, R26 to R212, R19 to R213, R20 to R214, R27 to R215, R28 to R216, U5 to U201, U8 to U202, U7 to U203, U9 to U203
Connections:
- wire segments 72 -> 60
