File: hardware/stm32-wifi-door-bell-input.sch (KiCad schematic (older format))
At the start: 23 parts, among them P201 FRONT, P202 BACK, U201 OPAMP-DUAL, U202 OPAMP-DUAL, U203 OPAMP-DUAL

Commit message: initial layout
Parts:
- U201, U202, U203: footprint (none) -> kicadlib:SOIC127P790X216-8N; MfgPartNumber (none) -> LM358PSR
Changed lines of the file:
@@
 $EndComp
 $Comp
-L GNDPWR #PWR013
+L GNDPWR #PWR014
 U 1 1 54B1A9EE
 P 1700 2400
-F 0 "#PWR013" H 1700 2450 40  0001 C CNN
+F 0 "#PWR014" H 1700 2450 40  0001 C CNN
 F 1 "GNDPWR" H 1700 2320 40  0001 C CNN
 F 2 "" H 1700 2400 60  0000 C CNN
@@
 F 0 "U201" H 3400 1750 60  0000 L CNN
 F 1 "OPAMP-DUAL" H 3400 1650 60  0000 L CNN
-F 2 "" H 3200 1900 60  0001 C CNN
+F 2 "kicadlib:SOIC127P790X216-8N" H 3200 1900 60  0001 C CNN
 F 3 "" H 3200 1900 60  0000 C CNN
+F 4 "LM358PSR" H 3200 1900 60  0001 C CNN "MfgPartNumber"
 	1    3200 1900
 	1    0    0    -1
@@
 F 0 "U201" H 4700 1850 60  0000 L CNN
 F 1 "OPAMP-DUAL" H 4700 1750 60  0000 L CNN
-F 2 "" H 4500 2000 60  0001 C CNN
+F 2 "kicadlib:SOIC127P790X216-8N" H 4500 2000 60  0001 C CNN
 F 3 "" H 4500 2000 60  0000 C CNN
+F 4 "LM358PSR" H 4500 2000 60  0001 C CNN "MfgPartNumber"
 	2    4500 2000
 	1    0    0    -1
@@
 $EndComp
 $Comp
-L GNDPWR #PWR014
+L GNDPWR #PWR015
 U 1 1 54B1AA1B
 P 3200 2600
-F 0 "#PWR014" H 3200 2650 40  0001 C CNN
+F 0 "#PWR015" H 3200 2650 40  0001 C CNN
 F 1 "GNDPWR" H 3200 2520 40  0001 C CNN
 F 2 "" H 3200 2600 60  0000 C CNN
@@
 	2400 2000 2300 2000
 $Comp
-L Vcc #PWR015
+L Vcc #PWR016
 U 1 1 54B1AA25
 P 3200 1400
-F 0 "#PWR015" H 3200 1490 20  0001 C CNN
+F 0 "#PWR016" H 3200 1490 20  0001 C CNN
 F 1 "Vcc" H 3200 1490 30  0000 C CNN
 F 2 "" H 3200 1400 60  0000 C CNN
@@
 	2700 1800 2700 2600
 $Comp
-L GNDPWR #PWR016
+L GNDPWR #PWR017
 U 1 1 54B1AA33
 P 2700 2600
-F 0 "#PWR016" H 2700 2650 40  0001 C CNN
+F 0 "#PWR017" H 2700 2650 40  0001 C CNN
 F 1 "GNDPWR" H 2700 2520 40  0001 C CNN
 F 2 "" H 2700 2600 60  0000 C CNN
@@
 Connection ~ 4100 2100
 $Comp
-L GNDPWR #PWR017
+L GNDPWR #PWR018
 U 1 1 54B1AA4B
 P 4100 2600
-F 0 "#PWR017" H 4100 2650 40  0001 C CNN
+F 0 "#PWR018" H 4100 2650 40  0001 C CNN
 F 1 "GNDPWR" H 4100 2520 40  0001 C CNN
 F 2 "" H 4100 2600 60  0000 C CNN
@@
 	4100 2400 4100 2600
 $Comp
-L Vcc #PWR018
+L Vcc #PWR019
 U 1 1 54B1AA52
 P 4100 1400
-F 0 "#PWR018" H 4100 1490 20  0001 C CNN
+F 0 "#PWR019" H 4100 1490 20  0001 C CNN
 F 1 "Vcc" H 4100 1490 30  0000 C CNN
 F 2 "" H 4100 1400 60  0000 C CNN
@@
 $EndComp
 $Comp
-L GNDPWR #PWR019
+L GNDPWR #PWR020
 U 1 1 54B1F484
 P 1700 4700
-F 0 "#PWR019" H 1700 4750 40  0001 C CNN
+F 0 "#PWR020" H 1700 4750 40  0001 C CNN
 F 1 "GNDPWR" H 1700 4620 40  0001 C CNN
 F 2 "" H 1700 4700 60  0000 C CNN
@@
 $EndComp
 $Comp
-L GNDPWR #PWR020
+L GNDPWR #PWR021
 U 1 1 54B1FBB7
 P 5400 2600
-F 0 "#PWR020" H 5400 2650 40  0001 C CNN
+F 0 "#PWR021" H 5400 2650 40  0001 C CNN
 F 1 "GNDPWR" H 5400 2520 40  0001 C CNN
 F 2 "" H 5400 2600 60  0000 C CNN
@@
 F 0 "U203" H 6400 1950 60  0000 L CNN
 F 1 "OPAMP-DUAL" H 6400 1850 60  0000 L CNN
-F 2 "" H 6200 2100 60  0001 C CNN
+F 2 "kicadlib:SOIC127P790X216-8N" H 6200 2100 60  0001 C CNN
 F 3 "" H 6200 2100 60  0000 C CNN
+F 4 "LM358PSR" H 6200 2100 60  0001 C CNN "MfgPartNumber"
 	1    6200 2100
 	1    0    0    -1
@@
 Connection ~ 5700 2200
 $Comp
-L GNDPWR #PWR021
+L GNDPWR #PWR022
 U 1 1 54B1FF14
 P 5700 2600
-F 0 "#PWR021" H 5700 2650 40  0001 C CNN
+F 0 "#PWR022" H 5700 2650 40  0001 C CNN
 F 1 "GNDPWR" H 5700 2520 40  0001 C CNN
 F 2 "" H 5700 2600 60  0000 C CNN
@@
 	5700 2500 5700 2600
 $Comp
-L Vcc #PWR022
+L Vcc #PWR023
 U 1 1 54B1FF62
 P 5700 1400
-F 0 "#PWR022" H 5700 1490 20  0001 C CNN
+F 0 "#PWR023" H 5700 1490 20  0001 C CNN
 F 1 "Vcc" H 5700 1490 30  0000 C CNN
 F 2 "" H 5700 1400 60  0000 C CNN
@@
 	5700 1400 5700 1700
 $Comp
-L GNDPWR #PWR023
+L GNDPWR #PWR024
 U 1 1 54B20160
 P 6200 2600
-F 0 "#PWR023" H 6200 2650 40  0001 C CNN
+F 0 "#PWR024" H 6200 2650 40  0001 C CNN
 F 1 "GNDPWR" H 6200 2520 40  0001 C CNN
 F 2 "" H 6200 2600 60  0000 C CNN
@@
 	6200 2400 6200 2600
 $Comp
-L +3.3V #PWR024
+L +3.3V #PWR025
 U 1 1 54B201A4
 P 6200 1400
-F 0 "#PWR024" H 6200 1490 20  0001 C CNN
+F 0 "#PWR025" H 6200 1490 20  0001 C CNN
 F 1 "+3.3V" H 6200 1490 30  0000 C CNN
 F 2 "" H 6200 1400 60  0000 C CNN
@@
 F 0 "U202" H 3400 4050 60  0000 L CNN
 F 1 "OPAMP-DUAL" H 3400 3950 60  0000 L CNN
-F 2 "" H 3200 4200 60  0001 C CNN
+F 2 "kicadlib:SOIC127P790X216-8N" H 3200 4200 60  0001 C CNN
 F 3 "" H 3200 4200 60  0000 C CNN
+F 4 "LM358PSR" H 3200 4200 60  0001 C CNN "MfgPartNumber"
 	1    3200 4200
 	1    0    0    -1
@@
 F 0 "U202" H 4700 4150 60  0000 L CNN
 F 1 "OPAMP-DUAL" H 4700 4050 60  0000 L CNN
-F 2 "" H 4500 4300 60  0001 C CNN
+F 2 "kicadlib:SOIC127P790X216-8N" H 4500 4300 60  0001 C CNN
 F 3 "" H 4500 4300 60  0000 C CNN
+F 4 "LM358PSR" H 4500 4300 60  0001 C CNN "MfgPartNumber"
 	2    4500 4300
 	1    0    0    -1
@@
 $EndComp
 $Comp
-L GNDPWR #PWR025
+L GNDPWR #PWR026
 U 1 1 54B20FC2
 P 3200 4900
-F 0 "#PWR025" H 3200 4950 40  0001 C CNN
+F 0 "#PWR026" H 3200 4950 40  0001 C CNN
 F 1 "GNDPWR" H 3200 4820 40  0001 C CNN
 F 2 "" H 3200 4900 60  0000 C CNN
@@
 Connection ~ 2800 4300
 $Comp
-L Vcc #PWR026
+L Vcc #PWR027
 U 1 1 54B20FCB
 P 3200 3700
-F 0 "#PWR026" H 3200 3790 20  0001 C CNN
+F 0 "#PWR027" H 3200 3790 20  0001 C CNN
 F 1 "Vcc" H 3200 3790 30  0000 C CNN
 F 2 "" H 3200 3700 60  0000 C CNN
@@
 	2700 4100 2700 4900
 $Comp
-L GNDPWR #PWR027
+L GNDPWR #PWR028
 U 1 1 54B20FD9
 P 2700 4900
-F 0 "#PWR027" H 2700 4950 40  0001 C CNN
+F 0 "#PWR028" H 2700 4950 40  0001 C CNN
 F 1 "GNDPWR" H 2700 4820 40  0001 C CNN
 F 2 "" H 2700 4900 60  0000 C CNN
@@
 Connection ~ 4100 4400
 $Comp
-L GNDPWR #PWR028
+L GNDPWR #PWR029
 U 1 1 54B20FEF
 P 4100 4900
-F 0 "#PWR028" H 4100 4950 40  0001 C CNN
+F 0 "#PWR029" H 4100 4950 40  0001 C CNN
 F 1 "GNDPWR" H 4100 4820 40  0001 C CNN
 F 2 "" H 4100 4900 60  0000 C CNN
@@
 	4100 4700 4100 4900
 $Comp
-L Vcc #PWR029
+L Vcc #PWR030
 U 1 1 54B20FF6
 P 4100 3700
-F 0 "#PWR029" H 4100 3790 20  0001 C CNN
+F 0 "#PWR030" H 4100 3790 20  0001 C CNN
 F 1 "Vcc" H 4100 3790 30  0000 C CNN
 F 2 "" H 4100 3700 60  0000 C CNN
@@
 $EndComp
 $Comp
-L GNDPWR #PWR030
+L GNDPWR #PWR031
 U 1 1 54B21009
 P 5400 4900
-F 0 "#PWR030" H 5400 4950 40  0001 C CNN
+F 0 "#PWR031" H 5400 4950 40  0001 C CNN
 F 1 "GNDPWR" H 5400 4820 40  0001 C CNN
 F 2 "" H 5400 4900 60  0000 C CNN
@@
 F 0 "U203" H 6400 4250 60  0000 L CNN
 F 1 "OPAMP-DUAL" H 6400 4150 60  0000 L CNN
-F 2 "" H 6200 4400 60  0001 C CNN
+F 2 "kicadlib:SOIC127P790X216-8N" H 6200 4400 60  0001 C CNN
 F 3 "" H 6200 4400 60  0000 C CNN
+F 4 "LM358PSR" H 6200 4400 60  0001 C CNN "MfgPartNumber"
 	2    6200 4400
 	1    0    0    -1
@@
 Connection ~ 5700 4500
 $Comp
-L GNDPWR #PWR031
+L GNDPWR #PWR032
 U 1 1 54B21029
 P 5700 4900
-F 0 "#PWR031" H 5700 4950 40  0001 C CNN
+F 0 "#PWR032" H 5700 4950 40  0001 C CNN
 F 1 "GNDPWR" H 5700 4820 40  0001 C CNN
 F 2 "" H 5700 4900 60  0000 C CNN
@@
 	5700 4800 5700 4900
 $Comp
-L Vcc #PWR032
+L Vcc #PWR033
 U 1 1 54B21030
 P 5700 3700
-F 0 "#PWR032" H 5700 3790 20  0001 C CNN
+F 0 "#PWR033" H 5700 3790 20  0001 C CNN
 F 1 "Vcc" H 5700 3790 30  0000 C CNN
 F 2 "" H 5700 3700 60  0000 C CNN

Commit message: clean up pcb
Parts:
- added P203: FRONT, kicadlib:HDRV1W66P254_1X1_254X249X838P, symbol P01
- added P204: BACK, kicadlib:HDRV1W66P254_1X1_254X249X838P, symbol P01
- P201, P202: footprint kicadlib:OST-OSTTC022162 -> kicadlib:OST-OSTTA024163
Connections:
- wire segments 60 -> 64

Commit message: v20150125
Parts:
- D201, D202: inventoryId (none) -> 273
- P201, P202: inventoryId (none) -> 603
- P203, P204: inventoryId (none) -> NA
- R201, R202, R203, R204, R205, R206, R207, R208, R214, R216: inventoryId (none) -> 454
- R209, R210: inventoryId (none) -> 613
- R211, R212: inventoryId (none) -> 532
- R213, R215: inventoryId (none) -> 299
- U201, U202, U203: inventoryId (none) -> 371
Changed lines of the file:
@@
 F 3 "" H 1300 1900 60  0000 C CNN
 F 4 "OSTTC022162" H 1300 1900 60  0001 C CNN "MfgPartNumber"
+F 5 "603" H 1300 1900 60  0001 C CNN "inventoryId"
 	1    1300 1900
 	-1   0    0    -1
@@
 F 3 "" H 3200 1900 60  0000 C CNN
 F 4 "LM358PSR" H 3200 1900 60  0001 C CNN "MfgPartNumber"
+F 5 "371" H 3200 1900 60  0001 C CNN "inventoryId"
 	1    3200 1900
 	1    0    0    -1
@@
 F 3 "" H 4500 2000 60  0000 C CNN
 F 4 "LM358PSR" H 4500 2000 60  0001 C CNN "MfgPartNumber"
+F 5 "371" H 4500 2000 60  0001 C CNN "inventoryId"
 	2    4500 2000
 	1    0    0    -1
@@
 F 2 "kicadlib:DIOM5226X220N" H 2200 2000 60  0001 C CNN
 F 3 "" H 2200 2000 60  0000 C CNN
+F 4 "273" H 2200 2000 60  0001 C CNN "inventoryId"
 	1    2200 2000
 	-1   0    0    1
@@
 F 2 "kicadlib:RESC2012X100N" H 2500 2000 60  0001 C CNN
 F 3 "" H 2500 2000 60  0000 C CNN
+F 4 "454" H 2500 2000 60  0001 C CNN "inventoryId"
 	1    2500 2000
 	0    -1   -1   0
@@
 F 2 "kicadlib:RESC2012X100N" H 3000 2400 60  0001 C CNN
 F 3 "" H 3000 2400 60  0000 C CNN
+F 4 "454" H 3000 2400 60  0001 C CNN "inventoryId"
 	1    3000 2400
 	0    -1   -1   0
@@
 F 2 "kicadlib:RESC2012X100N" H 4100 2300 60  0001 C CNN
 F 3 "" H 4100 2300 60  0000 C CNN
+F 4 "454" H 4100 2300 60  0001 C CNN "inventoryId"
 	1    4100 2300
 	1    0    0    -1
@@
 F 2 "kicadlib:RESC2012X100N" H 4100 1700 60  0001 C CNN
 F 3 "" H 4100 1700 60  0000 C CNN
+F 4 "454" H 4100 1700 60  0001 C CNN "inventoryId"
 	1    4100 1700
 	1    0    0    -1
@@
 F 3 "" H 1300 4200 60  0000 C CNN
 F 4 "OSTTC022162" H 1300 4200 60  0001 C CNN "MfgPartNumber"
+F 5 "603" H 1300 4200 60  0001 C CNN "inventoryId"
 	1    1300 4200
 	-1   0    0    -1
@@
 F 2 "kicadlib:RESC2012X100N" H 5200 2000 60  0001 C CNN
 F 3 "" H 5200 2000 60  0000 C CNN
+F 4 "613" H 5200 2000 60  0001 C CNN "inventoryId"
 	1    5200 2000
 	0    1    1    0
@@
 F 2 "kicadlib:RESC2012X100N" H 5400 2400 60  0001 C CNN
 F 3 "" H 5400 2400 60  0000 C CNN
+F 4 "532" H 5400 2400 60  0001 C CNN "inventoryId"
 	1    5400 2400
 	-1   0    0    1
@@
 F 3 "" H 6200 2100 60  0000 C CNN
 F 4 "LM358PSR" H 6200 2100 60  0001 C CNN "MfgPartNumber"
+F 5 "371" H 6200 2100 60  0001 C CNN "inventoryId"
 	1    6200 2100
 	1    0    0    -1
@@
 F 2 "kicadlib:RESC2012X100N" H 5700 2400 60  0001 C CNN
 F 3 "" H 5700 2400 60  0000 C CNN
+F 4 "454" H 5700 2400 60  0001 C CNN "inventoryId"
 	1    5700 2400
 	-1   0    0    1
@@
 F 2 "kicadlib:RESC2012X100N" H 5700 1800 60  0001 C CNN
 F 3 "" H 5700 1800 60  0000 C CNN
+F 4 "299" H 5700 1800 60  0001 C CNN "inventoryId"
 	1    5700 1800
 	-1   0    0    1
@@
 F 3 "" H 3200 4200 60  0000 C CNN
 F 4 "LM358PSR" H 3200 4200 60  0001 C CNN "MfgPartNumber"
+F 5 "371" H 3200 4200 60  0001 C CNN "inventoryId"
 	1    3200 4200
 	1    0    0    -1
@@
 F 3 "" H 4500 4300 60  0000 C CNN
 F 4 "LM358PSR" H 4500 4300 60  0001 C CNN "MfgPartNumber"
+F 5 "371" H 4500 4300 60  0001 C CNN "inventoryId"
 	2    4500 4300
 	1    0    0    -1
@@
 F 2 "kicadlib:RESC2012X100N" H 2500 4300 60  0001 C CNN
 F 3 "" H 2500 4300 60  0000 C CNN
+F 4 "454" H 2500 4300 60  0001 C CNN "inventoryId"
 	1    2500 4300
 	0    -1   -1   0
@@
 F 2 "kicadlib:RESC2012X100N" H 3000 4700 60  0001 C CNN
 F 3 "" H 3000 4700 60  0000 C CNN
+F 4 "454" H 3000 4700 60  0001 C CNN "inventoryId"
 	1    3000 4700
 	0    -1   -1   0
@@
 F 2 "kicadlib:RESC2012X100N" H 4100 4600 60  0001 C CNN
 F 3 "" H 4100 4600 60  0000 C CNN
+F 4 "454" H 4100 4600 60  0001 C CNN "inventoryId"
 	1    4100 4600
 	1    0    0    -1
@@
 F 2 "kicadlib:RESC2012X100N" H 4100 4000 60  0001 C CNN
 F 3 "" H 4100 4000 60  0000 C CNN
+F 4 "454" H 4100 4000 60  0001 C CNN "inventoryId"
 	1    4100 4000
 	1    0    0    -1
@@
 F 2 "kicadlib:RESC2012X100N" H 5200 4300 60  0001 C CNN
 F 3 "" H 5200 4300 60  0000 C CNN
+F 4 "613" H 5200 4300 60  0001 C CNN "inventoryId"
 	1    5200 4300
 	0    1    1    0
@@
 F 2 "kicadlib:RESC2012X100N" H 5400 4700 60  0001 C CNN
 F 3 "" H 5400 4700 60  0000 C CNN
+F 4 "532" H 5400 4700 60  0001 C CNN "inventoryId"
 	1    5400 4700
 	-1   0    0    1
@@
 F 3 "" H 6200 4400 60  0000 C CNN
 F 4 "LM358PSR" H 6200 4400 60  0001 C CNN "MfgPartNumber"
+F 5 "371" H 6200 4400 60  0001 C CNN "inventoryId"
 	2    6200 4400
 	1    0    0    -1
@@
 F 2 "kicadlib:RESC2012X100N" H 5700 4700 60  0001 C CNN
 F 3 "" H 5700 4700 60  0000 C CNN
+F 4 "454" H 5700 4700 60  0001 C CNN "inventoryId"
 	1    5700 4700
 	-1   0    0    1
@@
 F 2 "kicadlib:RESC2012X100N" H 5700 4100 60  0001 C CNN
 F 3 "" H 5700 4100 60  0000 C CNN
+F 4 "299" H 5700 4100 60  0001 C CNN "inventoryId"
 	1    5700 4100
 	-1   0    0    1
@@
 F 2 "kicadlib:DIOM5226X220N" H 2200 4300 60  0001 C CNN
 F 3 "" H 2200 4300 60  0000 C CNN
+F 4 "273" H 2200 4300 60  0001 C CNN "inventoryId"
 	1    2200 4300
 	-1   0    0    1
@@
 F 2 "kicadlib:HDRV1W66P254_1X1_254X249X838P" H 7150 1600 60  0001 C CNN
 F 3 "" H 7150 1600 60  0000 C CNN
+F 4 "NA" H 7150 1600 60  0001 C CNN "inventoryId"
 	1    7150 1600
 	1    0    0    -1
@@
 F 2 "kicadlib:HDRV1W66P254_1X1_254X249X838P" H 7150 3900 60  0001 C CNN
 F 3 "" H 7150 3900 60  0000 C CNN
+F 4 "NA" H 7150 3900 60  0001 C CNN "inventoryId"
 	1    7150 3900
 	1    0    0    -1

Commit message: door bell button schematic
Parts:
- P201: MfgPartNumber OSTTC022162 -> (none)
Changed lines of the file:
@@
 F 2 "kicadlib:OST-OSTTA024163" H 1300 1900 60  0001 C CNN
 F 3 "" H 1300 1900 60  0000 C CNN
-F 4 "OSTTC022162" H 1300 1900 60  0001 C CNN "MfgPartNumber"
-F 5 "603" H 1300 1900 60  0001 C CNN "inventoryId"
+F 4 "603" H 1300 1900 60  0001 C CNN "inventoryId"
 	1    1300 1900
 	-1   0    0    -1
