File: hardware/$stm32-wifi-door-bell-input.sch (KiCad schematic (older format))
At the start: 23 parts, among them P201 FRONT, P202 BACK, U201 OPAMP-DUAL, U202 OPAMP-DUAL, U203 OPAMP-DUAL

Commit message: more schematics
Parts:
- U201, U202, U203: MfgPartNumber (none) -> LM358PSR
Changed lines of the file:
@@
 F 2 "" H 3200 1900 60  0001 C CNN
 F 3 "" H 3200 1900 60  0000 C CNN
+F 4 "LM358PSR" H 3200 1900 60  0001 C CNN "MfgPartNumber"
 	1    3200 1900
 	1    0    0    -1
@@
 F 2 "" H 4500 2000 60  0001 C CNN
 F 3 "" H 4500 2000 60  0000 C CNN
+F 4 "LM358PSR" H 4500 2000 60  0001 C CNN "MfgPartNumber"
 	2    4500 2000
 	1    0    0    -1
@@
 F 2 "" H 6200 2100 60  0001 C CNN
 F 3 "" H 6200 2100 60  0000 C CNN
+F 4 "LM358PSR" H 6200 2100 60  0001 C CNN "MfgPartNumber"
 	1    6200 2100
 	1    0    0    -1
@@
 F 2 "" H 3200 4200 60  0001 C CNN
 F 3 "" H 3200 4200 60  0000 C CNN
+F 4 "LM358PSR" H 3200 4200 60  0001 C CNN "MfgPartNumber"
 	1    3200 4200
 	1    0    0    -1
@@
 F 2 "" H 4500 4300 60  0001 C CNN
 F 3 "" H 4500 4300 60  0000 C CNN
+F 4 "LM358PSR" H 4500 4300 60  0001 C CNN "MfgPartNumber"
 	2    4500 4300
 	1    0    0    -1
@@
 F 2 "" H 6200 4400 60  0001 C CNN
 F 3 "" H 6200 4400 60  0000 C CNN
+F 4 "LM358PSR" H 6200 4400 60  0001 C CNN "MfgPartNumber"
 	2    6200 4400
 	1    0    0    -1
