File: hardware/stm32-wifi-door-bell.sch (KiCad schematic (older format))
At the start: 31 parts, among them J1 USB, P1 SWD, P2 FTDI-PLUG, U1 STM32-48PIN, X1 32.768kHz, X2 8MHz

Commit message: update schematic
Parts:
- added BT1: BATTERY, symbol BATTERY
- added R4, R6, R7: 10K, kicadlib:RESC2012X100N, symbol R
- U1: value STM32-48PIN -> STM32F072CBT6
- gave numbers to parts that had none: 11
Connections:
- net labels added: BTNBACK, BTNFRONT, DACOUT
- wire segments 152 -> 168
- no-connect marks 9 -> 21
Other:
- moved on the sheet: C1, C10, C11, C12, C13, C14, C17, C18, C2, C3, C4, C5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

Commit message: more schematic work
Parts:
- removed C12: 1uF, kicadlib:CAPC2012X100N, symbol C
- removed C13, C14: 0.1uF, kicadlib:CAPC2012X100N, symbol C
- removed C17: 10pF, kicadlib:CAPC2012X100N, symbol C
- removed C18: 2.2pF, kicadlib:CAPC2012X100N, symbol C
- removed L2: 2.2nH, symbol INDUCTOR
- removed L3: DNP, symbol INDUCTOR
- removed P3: P03, symbol P03
- removed R4, R6, R7: 10K, kicadlib:RESC2012X100N, symbol R
- removed U2: MICROSD-AMPHENOL-114-00841-68, symbol MICROSD-AMPHENOL-114-00841-68
- removed U3: TICC3000, symbol TICC3000
- removed X3: ANT, symbol ANT
Connections:
- net labels removed: CC3000RX, CC3000TX
- wire segments 168 -> 129
- no-connect marks 21 -> 15
Other:
- moved on the sheet: C1, C10, C11, C2, C3, C4, C5, C6, C7, C8, C9, J1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

Commit message: reannotate schematic
Parts:
- renumbered BT1 to BT101, C7 to C101, C8 to C102, C9 to C103, C1 to C104, C10 to C105, C2 to C106, C11 to C107, C3 to C108, C4 to C109, C5 to C110, C6 to C111, J1 to J101, P1 to P101, P2 to P102, R1 to R101, R2 to R102, R3 to R103, U1 to U101, X1 to X101, X2 to X102
Changed lines of the file:
@@
 $EndDescr
 $Comp
-L STM32-48PIN U1
+L STM32-48PIN U101
 U 1 1 5488778C
 P 4400 3400
-F 0 "U1" H 3800 5150 60  0000 C CNN
+F 0 "U101" H 3800 5150 60  0000 C CNN
 F 1 "STM32F072CBT6" H 3750 1650 60  0000 L CNN
 F 2 "kicadlib:QFP50P900X900X160-48N" H 4400 3400 60  0001 C CNN
@@
 $EndComp
 $Comp
-L GNDPWR #PWR12
+L GNDPWR #PWR111
 U 1 1 54887804
 P 3350 5100
-F 0 "#PWR12" H 3350 5150 40  0001 C CNN
+F 0 "#PWR111" H 3350 5150 40  0001 C CNN
 F 1 "GNDPWR" H 3350 5020 40  0001 C CNN
 F 2 "" H 3350 5100 60  0000 C CNN
@@
 $EndComp
 $Comp
-L SWD P1
+L SWD P101
 U 1 1 5488788C
 P 3700 7300
-F 0 "P1" H 3700 7950 60  0000 L CNN
+F 0 "P101" H 3700 7950 60  0000 L CNN
 F 1 "SWD" H 3700 7150 60  0000 L CNN
 F 2 "kicadlib:HDRV6W66P254_1X6_1524X249X838P" H 3400 7200 60  0001 C CNN
@@
 $EndComp
 $Comp
-L FTDI-PLUG P2
+L FTDI-PLUG P102
 U 1 1 54887927
 P 5600 7300
-F 0 "P2" H 5600 7950 60  0000 L CNN
+F 0 "P102" H 5600 7950 60  0000 L CNN
 F 1 "FTDI-PLUG" H 5600 7150 60  0000 L CNN
 F 2 "kicadlib:HDRV6W66P254_1X6_1524X249X838P" H 5600 7100 60  0001 C CNN
@@
 $EndComp
 $Comp
-L GNDPWR #PWR4
+L GNDPWR #PWR109
 U 1 1 548879DB
 P 3300 7400
-F 0 "#PWR4" H 3300 7450 40  0001 C CNN
+F 0 "#PWR109" H 3300 7450 40  0001 C CNN
 F 1 "GNDPWR" H 3300 7320 40  0001 C CNN
 F 2 "" H 3300 7400 60  0000 C CNN
@@
 $EndComp
 $Comp
-L GNDPWR #PWR5
+L GNDPWR #PWR112
 U 1 1 548879EF
 P 5200 7400
-F 0 "#PWR5" H 5200 7450 40  0001 C CNN
+F 0 "#PWR112" H 5200 7450 40  0001 C CNN
 F 1 "GNDPWR" H 5200 7320 40  0001 C CNN
 F 2 "" H 5200 7400 60  0000 C CNN
@@
 $EndComp
 $Comp
-L +3.3V #PWR11
+L +3.3V #PWR110
 U 1 1 54887A2E
 P 3350 1700
-F 0 "#PWR11" H 3350 1790 20  0001 C CNN
+F 0 "#PWR110" H 3350 1790 20  0001 C CNN
 F 1 "+3.3V" H 3350 1790 30  0000 C CNN
 F 2 "" H 3350 1700 60  0000 C CNN
@@
 $EndComp
 $Comp
-L CRYSTAL-14 X1
+L CRYSTAL-14 X101
 U 1 1 5488786B
 P 3350 2650
-F 0 "X1" H 3350 2725 30  0000 C CNN
+F 0 "X101" H 3350 2725 30  0000 C CNN
 F 1 "32.768kHz" H 3350 2570 30  0000 C CNN
 F 2 "kicadlib:SOJ550P370X240-4N" H 3350 2650 60  0001 C CNN
@@
 $EndComp
 $Comp
-L CRYSTAL X2
+L CRYSTAL X102
 U 1 1 5488789E
 P 3350 3350
-F 0 "X2" H 3350 3425 30  0000 C CNN
+F 0 "X102" H 3350 3425 30  0000 C CNN
 F 1 "8MHz" H 3350 3270 30  0000 C CNN
 F 2 "kicadlib:XTAL8045X200N" H 3350 3350 60  0001 C CNN
@@
 $EndComp
 $Comp
-L C C6
+L C C111
 U 1 1 548878C1
 P 3150 3600
-F 0 "C6" H 3175 3650 30  0000 L CNN
+F 0 "C111" H 3175 3650 30  0000 L CNN
 F 1 "18pF" H 3175 3550 30  0000 L CNN
 F 2 "kicadlib:CAPC2012X100N" H 3150 3600 60  0001 C CNN
@@
 $EndComp
 $Comp
-L C C5
+L C C110
 U 1 1 548878EE
 P 3150 3100
-F 0 "C5" H 3175 3150 30  0000 L CNN
+F 0 "C110" H 3175 3150 30  0000 L CNN
 F 1 "18pF" H 3175 3050 30  0000 L CNN
 F 2 "kicadlib:CAPC2012X100N" H 3150 3100 60  0001 C CNN
@@
 $EndComp
 $Comp
-L C C4
+L C C109
 U 1 1 5488791D
 P 3150 2900
-F 0 "C4" H 3175 2950 30  0000 L CNN
+F 0 "C109" H 3175 2950 30  0000 L CNN
 F 1 "18pF" H 3175 2850 30  0000 L CNN
 F 2 "kicadlib:CAPC2012X100N" H 3150 2900 60  0001 C CNN
@@
 $EndComp
 $Comp
-L C C3
+L C C108
 U 1 1 5488793D
 P 3150 2400
-F 0 "C3" H 3175 2450 30  0000 L CNN
+F 0 "C108" H 3175 2450 30  0000 L CNN
 F 1 "18pF" H 3175 2350 30  0000 L CNN
 F 2 "kicadlib:CAPC2012X100N" H 3150 2400 60  0001 C CNN
@@
 $EndComp
 $Comp
-L GNDPWR #PWR10
+L GNDPWR #PWR107
 U 1 1 548879FD
 P 2850 3700
-F 0 "#PWR10" H 2850 3750 40  0001 C CNN
+F 0 "#PWR107" H 2850 3750 40  0001 C CNN
 F 1 "GNDPWR" H 2850 3620 40  0001 C CNN
 F 2 "" H 2850 3700 60  0000 C CNN
@@
 SWDIO
 $Comp
-L +3.3V #PWR3
+L +3.3V #PWR108
 U 1 1 54887EAF
 P 3300 6700
-F 0 "#PWR3" H 3300 6790 20  0001 C CNN
+F 0 "#PWR108" H 3300 6790 20  0001 C CNN
 F 1 "+3.3V" H 3300 6790 30  0000 C CNN
 F 2 "" H 3300 6700 60  0000 C CNN
@@
 DEBUGTX
 $Comp
-L C C2
+L C C106
 U 1 1 548881C8
 P 2650 4200
-F 0 "C2" H 2675 4250 30  0000 L CNN
+F 0 "C106" H 2675 4250 30  0000 L CNN
 F 1 "47pF" H 2675 4150 30  0000 L CNN
 F 2 "kicadlib:CAPC2012X100N" H 2650 4200 60  0001 C CNN
@@
 $EndComp
 $Comp
-L C C1
+L C C104
 U 1 1 54888245
 P 2450 4200
-F 0 "C1" H 2475 4250 30  0000 L CNN
+F 0 "C104" H 2475 4250 30  0000 L CNN
 F 1 "47pF" H 2475 4150 30  0000 L CNN
 F 2 "kicadlib:CAPC2012X100N" H 2450 4200 60  0001 C CNN
@@
 $EndComp
 $Comp
-L GNDPWR #PWR9
+L GNDPWR #PWR106
 U 1 1 54888276
 P 2450 4500
-F 0 "#PWR9" H 2450 4550 40  0001 C CNN
+F 0 "#PWR106" H 2450 4550 40  0001 C CNN
 F 1 "GNDPWR" H 2450 4420 40  0001 C CNN
 F 2 "" H 2450 4500 60  0000 C CNN
@@
 $EndComp
 $Comp
-L R R2
+L R R102
 U 1 1 5488849C
 P 2250 3900
-F 0 "R2" V 2195 3900 30  0000 C CNN
+F 0 "R102" V 2195 3900 30  0000 C CNN
 F 1 "22R" V 2150 3900 30  0000 C CNN
 F 2 "kicadlib:RESC2012X100N" H 2250 3900 60  0001 C CNN
@@
 $EndComp
 $Comp
-L R R3
+L R R103
 U 1 1 548884EB
 P 2250 4000
-F 0 "R3" V 2350 4000 30  0000 C CNN
+F 0 "R103" V 2350 4000 30  0000 C CNN
 F 1 "22R" V 2305 4000 30  0000 C CNN
 F 2 "kicadlib:RESC2012X100N" H 2250 4000 60  0001 C CNN
@@
 USBDM
 $Comp
-L R R1
+L R R101
 U 1 1 548889AA
 P 2050 3600
-F 0 "R1" V 1995 3600 30  0000 C CNN
+F 0 "R101" V 1995 3600 30  0000 C CNN
 F 1 "1.5K" V 2105 3600 30  0000 C CNN
 F 2 "kicadlib:RESC2012X100N" H 2050 3600 60  0001 C CNN
@@
 USBDPPU
 $Comp
-L USB J1
+L USB J101
 U 1 1 54887F2F
 P 1800 7000
-F 0 "J1" H 1450 7350 60  0000 L CNN
+F 0 "J101" H 1450 7350 60  0000 L CNN
 F 1 "USB" H 1450 6650 60  0000 L CNN
 F 2 "kicadlib:JST_UB-MC5BR3-SD204-4S-NMP" H 1750 7000 60  0001 C CNN
@@
 $EndComp
 $Comp
-L GNDPWR #PWR8
+L GNDPWR #PWR104
 U 1 1 5488802A
 P 2100 7300
-F 0 "#PWR8" H 2100 7350 40  0001 C CNN
+F 0 "#PWR104" H 2100 7350 40  0001 C CNN
 F 1 "GNDPWR" H 2100 7220 40  0001 C CNN
 F 2 "" H 2100 7300 60  0000 C CNN
@@
 USBDM
 $Comp
-L +5V #PWR7
+L +5V #PWR103
 U 1 1 54888150
 P 2100 6700
-F 0 "#PWR7" H 2100 6790 20  0001 C CNN
+F 0 "#PWR103" H 2100 6790 20  0001 C CNN
 F 1 "+5V" H 2100 6790 30  0000 C CNN
 F 2 "" H 2100 6700 60  0000 C CNN
@@
 $EndComp
 $Comp
-L C C7
+L C C101
 U 1 1 548884DC
 P 1950 1900
-F 0 "C7" H 1975 1950 30  0000 L CNN
+F 0 "C101" H 1975 1950 30  0000 L CNN
 F 1 "0.1uF" H 1975 1850 30  0000 L CNN
 F 2 "kicadlib:CAPC2012X100N" H 1950 1900 60  0001 C CNN
@@
 $EndComp
 $Comp
-L C C8
+L C C102
 U 1 1 54888544
 P 2150 1900
-F 0 "C8" H 2175 1950 30  0000 L CNN
+F 0 "C102" H 2175 1950 30  0000 L CNN
 F 1 "0.1uF" H 2175 1850 30  0000 L CNN
 F 2 "kicadlib:CAPC2012X100N" H 2150 1900 60  0001 C CNN
@@
 $EndComp
 $Comp
-L C C9
+L C C103
 U 1 1 54888583
 P 2350 1900
-F 0 "C9" H 2375 1950 30  0000 L CNN
+F 0 "C103" H 2375 1950 30  0000 L CNN
 F 1 "0.1uF" H 2375 1850 30  0000 L CNN
 F 2 "kicadlib:CAPC2012X100N" H 2350 1900 60  0001 C CNN
@@
 $EndComp
 $Comp
-L C C10
+L C C105
 U 1 1 548885AD
 P 2550 1900
-F 0 "C10" H 2575 1950 30  0000 L CNN
+F 0 "C105" H 2575 1950 30  0000 L CNN
 F 1 "0.1uF" H 2575 1850 30  0000 L CNN
 F 2 "kicadlib:CAPC2012X100N" H 2550 1900 60  0001 C CNN
@@
 $EndComp
 $Comp
-L GNDPWR #PWR2
+L GNDPWR #PWR102
 U 1 1 54888615
 P 1950 2100
-F 0 "#PWR2" H 1950 2150 40  0001 C CNN
+F 0 "#PWR102" H 1950 2150 40  0001 C CNN
 F 1 "GNDPWR" H 1950 2020 40  0001 C CNN
 F 2 "" H 1950 2100 60  0000 C CNN
@@
 $EndComp
 $Comp
-L +3.3V #PWR1
+L +3.3V #PWR101
 U 1 1 5488867C
 P 1950 1700
-F 0 "#PWR1" H 1950 1790 20  0001 C CNN
+F 0 "#PWR101" H 1950 1790 20  0001 C CNN
 F 1 "+3.3V" H 1950 1790 30  0000 C CNN
 F 2 "" H 1950 1700 60  0000 C CNN
@@
 $EndComp
 $Comp
-L C C11
+L C C107
 U 1 1 54888B9A
 P 2750 1900
-F 0 "C11" H 2775 1950 30  0000 L CNN
+F 0 "C107" H 2775 1950 30  0000 L CNN
 F 1 "0.1uF" H 2775 1850 30  0000 L CNN
 F 2 "kicadlib:CAPC2012X100N" H 2750 1900 60  0001 C CNN
@@
 NoConn ~ 5400 5000
 $Comp
-L BATTERY BT1
+L BATTERY BT101
 U 1 1 54B165FC
 P 2350 2700
-F 0 "BT1" H 2350 2900 50  0000 C CNN
+F 0 "BT101" H 2350 2900 50  0000 C CNN
 F 1 "BATTERY" H 2350 2510 50  0000 C CNN
 F 2 "" H 2350 2700 60  0000 C CNN
@@
 $EndComp
 $Comp
-L GNDPWR #PWR6
+L GNDPWR #PWR105
 U 1 1 54B169FB
 P 2350 3100
-F 0 "#PWR6" H 2350 3150 40  0001 C CNN
+F 0 "#PWR105" H 2350 3150 40  0001 C CNN
 F 1 "GNDPWR" H 2350 3020 40  0001 C CNN
 F 2 "" H 2350 3100 60  0000 C CNN

Commit message: more schematics
Parts:
- added M101, M102, M103, M104: Mounting Hole, kicadlib:MTGNP565H328Z565P, symbol MECH
- BT101: footprint (none) -> kicadlib:KEYSTONE-3000
Connections:
- wire segments 129 -> 103
Changed lines of the file:
@@
 $EndComp
 $Comp
-L GNDPWR #PWR111
+L GNDPWR #PWR01
 U 1 1 54887804
 P 3350 5100
-F 0 "#PWR111" H 3350 5150 40  0001 C CNN
+F 0 "#PWR01" H 3350 5150 40  0001 C CNN
 F 1 "GNDPWR" H 3350 5020 40  0001 C CNN
 F 2 "" H 3350 5100 60  0000 C CNN
@@
 $EndComp
 $Comp
-L GNDPWR #PWR109
+L GNDPWR #PWR02
 U 1 1 548879DB
 P 3300 7400
-F 0 "#PWR109" H 3300 7450 40  0001 C CNN
+F 0 "#PWR02" H 3300 7450 40  0001 C CNN
 F 1 "GNDPWR" H 3300 7320 40  0001 C CNN
 F 2 "" H 3300 7400 60  0000 C CNN
@@
 $EndComp
 $Comp
-L GNDPWR #PWR112
+L GNDPWR #PWR03
 U 1 1 548879EF
 P 5200 7400
-F 0 "#PWR112" H 5200 7450 40  0001 C CNN
+F 0 "#PWR03" H 5200 7450 40  0001 C CNN
 F 1 "GNDPWR" H 5200 7320 40  0001 C CNN
 F 2 "" H 5200 7400 60  0000 C CNN
@@
 $EndComp
 $Comp
-L +3.3V #PWR110
+L +3.3V #PWR04
 U 1 1 54887A2E
 P 3350 1700
-F 0 "#PWR110" H 3350 1790 20  0001 C CNN
+F 0 "#PWR04" H 3350 1790 20  0001 C CNN
 F 1 "+3.3V" H 3350 1790 30  0000 C CNN
 F 2 "" H 3350 1700 60  0000 C CNN
@@
 $EndComp
 $Comp
-L GNDPWR #PWR107
+L GNDPWR #PWR05
 U 1 1 548879FD
 P 2850 3700
-F 0 "#PWR107" H 2850 3750 40  0001 C CNN
+F 0 "#PWR05" H 2850 3750 40  0001 C CNN
 F 1 "GNDPWR" H 2850 3620 40  0001 C CNN
 F 2 "" H 2850 3700 60  0000 C CNN
@@
 SWDIO
 $Comp
-L +3.3V #PWR108
+L +3.3V #PWR06
 U 1 1 54887EAF
 P 3300 6700
-F 0 "#PWR108" H 3300 6790 20  0001 C CNN
+F 0 "#PWR06" H 3300 6790 20  0001 C CNN
 F 1 "+3.3V" H 3300 6790 30  0000 C CNN
 F 2 "" H 3300 6700 60  0000 C CNN
@@
 $EndComp
 $Comp
-L GNDPWR #PWR106
+L GNDPWR #PWR07
 U 1 1 54888276
 P 2450 4500
-F 0 "#PWR106" H 2450 4550 40  0001 C CNN
+F 0 "#PWR07" H 2450 4550 40  0001 C CNN
 F 1 "GNDPWR" H 2450 4420 40  0001 C CNN
 F 2 "" H 2450 4500 60  0000 C CNN
@@
 $EndComp
 $Comp
-L GNDPWR #PWR104
+L GNDPWR #PWR08
 U 1 1 5488802A
 P 2100 7300
-F 0 "#PWR104" H 2100 7350 40  0001 C CNN
+F 0 "#PWR08" H 2100 7350 40  0001 C CNN
 F 1 "GNDPWR" H 2100 7220 40  0001 C CNN
 F 2 "" H 2100 7300 60  0000 C CNN
@@
 USBDM
 $Comp
-L +5V #PWR103
+L +5V #PWR09
 U 1 1 54888150
 P 2100 6700
-F 0 "#PWR103" H 2100 6790 20  0001 C CNN
+F 0 "#PWR09" H 2100 6790 20  0001 C CNN
 F 1 "+5V" H 2100 6790 30  0000 C CNN
 F 2 "" H 2100 6700 60  0000 C CNN
@@
 $EndComp
 $Comp
-L GNDPWR #PWR102
+L GNDPWR #PWR010
 U 1 1 54888615
 P 1950 2100
-F 0 "#PWR102" H 1950 2150 40  0001 C CNN
+F 0 "#PWR010" H 1950 2150 40  0001 C CNN
 F 1 "GNDPWR" H 1950 2020 40  0001 C CNN
 F 2 "" H 1950 2100 60  0000 C CNN
@@
 $EndComp
 $Comp
-L +3.3V #PWR101
+L +3.3V #PWR011
 U 1 1 5488867C
 P 1950 1700
-F 0 "#PWR101" H 1950 1790 20  0001 C CNN
+F 0 "#PWR011" H 1950 1790 20  0001 C CNN
 F 1 "+3.3V" H 1950 1790 30  0000 C CNN
 F 2 "" H 1950 1700 60  0000 C CNN
@@
 $EndSheet
 $Sheet
-S 9300 2100 600  200
+S 9300 2100 600  300
 U 54B1B30C
 F0 "power" 60
 F1 "stm32-wifi-door-bell-power.sch" 60
 F2 "FRONTIN" I L 9300 2200 60
+F3 "BACKIN" I L 9300 2300 60
 $EndSheet
 Text Label 8800 2400 2    60   ~ 0
@@
 F 0 "BT101" H 2350 2900 50  0000 C CNN
 F 1 "BATTERY" H 2350 2510 50  0000 C CNN
-F 2 "" H 2350 2700 60  0000 C CNN
+F 2 "kicadlib:KEYSTONE-3000" H 2350 2700 60  0001 C CNN
 F 3 "" H 2350 2700 60  0000 C CNN
 	1    2350 2700
@@
 $EndComp
 $Comp
-L GNDPWR #PWR105
+L GNDPWR #PWR012
 U 1 1 54B169FB
 P 2350 3100
-F 0 "#PWR105" H 2350 3150 40  0001 C CNN
+F 0 "#PWR012" H 2350 3150 40  0001 C CNN
 F 1 "GNDPWR" H 2350 3020 40  0001 C CNN
 F 2 "" H 2350 3100 60  0000 C CNN
@@
 	3450 4700 3350 4700
 Wire Wire Line
-	3350 4500 3350 4700
-Wire Wire Line
-	3350 4700 3350 4800
-Wire Wire Line
-	3350 4800 3350 4900
-Wire Wire Line
-	3350 4900 3350 5000
-Wire Wire Line
-	3350 5000 3350 5100
+	3350 4500 3350 5100
 Wire Wire Line
 	3450 4800 3350 4800
@@
 	3350 2100 3450 2100
 Wire Wire Line
-	3350 1700 3350 1800
-Wire Wire Line
-	3350 1800 3350 1900
-Wire Wire Line
-	3350 1900 3350 2000
-Wire Wire Line
-	3350 2000 3350 2100
+	3350 1700 3350 2100
 Wire Wire Line
 	3450 2000 3350 2000
@@
 	3050 2400 2850 2400
 Wire Wire Line
-	2850 2400 2850 2900
-Wire Wire Line
-	2850 2900 2850 3100
-Wire Wire Line
-	2850 3100 2850 3600
-Wire Wire Line
-	2850 3600 2850 3700
+	2850 2400 2850 3700
 Wire Wire Line
 	3050 2900 2850 2900
@@
 Connection ~ 2850 3600
 Wire Wire Line
-	3250 3600 3350 3600
-Wire Wire Line
-	3350 3600 3450 3600
-Wire Wire Line
-	3250 3100 3350 3100
-Wire Wire Line
-	3350 3100 3450 3100
-Wire Wire Line
-	3250 2900 3350 2900
-Wire Wire Line
-	3350 2900 3450 2900
-Wire Wire Line
-	3250 2400 3350 2400
-Wire Wire Line
-	3350 2400 3450 2400
+	3250 3600 3450 3600
+Wire Wire Line
+	3250 3100 3450 3100
+Wire Wire Line
+	3250 2900 3450 2900
+Wire Wire Line
+	3250 2400 3450 2400
 Wire Wire Line
 	3350 2500 3350 2400
@@
 	4700 7200 5300 7200
 Wire Wire Line
-	2450 4300 2450 4400
-Wire Wire Line
-	2450 4400 2450 4500
+	2450 4300 2450 4500
 Wire Wire Line
 	2650 4300 2650 4400
@@
 Connection ~ 2450 4400
 Wire Wire Line
-	2350 4000 2650 4000
-Wire Wire Line
-	2650 4000 3450 4000
+	2350 4000 3450 4000
 Wire Wire Line
 	2650 4000 2650 4100
 Wire Wire Line
-	2350 3900 2450 3900
-Wire Wire Line
-	2450 3900 3450 3900
+	2350 3900 3450 3900
 Wire Wire Line
 	2450 3900 2450 4100
@@
 Connection ~ 2450 3900
 Wire Wire Line
-	1450 3900 2050 3900
-Wire Wire Line
-	2050 3900 2150 3900
+	1450 3900 2150 3900
 Wire Wire Line
 	2150 4000 1450 4000
@@
 	2000 7200 2100 7200
 Wire Wire Line
-	2100 7100 2100 7200
-Wire Wire Line
-	2100 7200 2100 7300
+	2100 7100 2100 7300
 Wire Wire Line
 	2000 7100 2100 7100
@@
 	2000 7000 2400 7000
 Wire Wire Line
-	1950 1700 1950 1750
-Wire Wire Line
-	1950 1750 1950 1800
+	1950 1700 1950 1800
 Wire Wire Line
 	2550 1750 2550 1800
 Wire Wire Line
-	1950 1750 2150 1750
-Wire Wire Line
-	2150 1750 2350 1750
-Wire Wire Line
-	2350 1750 2550 1750
-Wire Wire Line
-	2550 1750 2750 1750
+	1950 1750 2750 1750
 Connection ~ 1950 1750
 Wire Wire Line
@@
 Connection ~ 2350 1750
 Wire Wire Line
-	1950 2000 1950 2050
-Wire Wire Line
-	1950 2050 1950 2100
-Wire Wire Line
-	1950 2050 2150 2050
-Wire Wire Line
-	2150 2050 2350 2050
-Wire Wire Line
-	2350 2050 2550 2050
-Wire Wire Line
-	2550 2050 2750 2050
+	1950 2000 1950 2100
+Wire Wire Line
+	1950 2050 2750 2050
 Wire Wire Line
 	2550 2050 2550 2000
@@
 Wire Wire Line
 	9300 4100 8800 4100
+Wire Wire Line
+	8200 2300 9300 2300
+$Comp
+L MECH M101
+U 1 1 54B5E845
+P 8800 5900
+F 0 "M101" H 8850 5900 60  0000 C CNN
+F 1 "Mounting Hole" H 9000 5900 60  0000 L CNN
+F 2 "kicadlib:MTGNP565H328Z565P" H 8800 5900 60  0001 C CNN
+F 3 "" H 8800 5900 60  0000 C CNN
+	1    8800 5900
+	1    0    0    -1
+$EndComp
+$Comp
+L MECH M102
+U 1 1 54B5EE87
+P 8800 6000
+F 0 "M102" H 8850 6000 60  0000 C CNN
+F 1 "Mounting Hole" H 9000 6000 60  0000 L CNN
+F 2 "kicadlib:MTGNP565H328Z565P" H 8800 6000 60  0001 C CNN
+F 3 "" H 8800 6000 60  0000 C CNN
+	1    8800 6000
+	1    0    0    -1
+$EndComp
+$Comp
+L MECH M103
+U 1 1 54B5EEB2
+P 8800 6100
+F 0 "M103" H 8850 6100 60  0000 C CNN
+F 1 "Mounting Hole" H 9000 6100 60  0000 L CNN
+F 2 "kicadlib:MTGNP565H328Z565P" H 8800 6100 60  0001 C CNN
+F 3 "" H 8800 6100 60  0000 C CNN
+	1    8800 6100
+	1    0    0    -1
+$EndComp
+$Comp
+L MECH M104
+U 1 1 54B5EEDE
+P 8800 6200
+F 0 "M104" H 8850 6200 60  0000 C CNN
+F 1 "Mounting Hole" H 9000 6200 60  0000 L CNN
+F 2 "kicadlib:MTGNP565H328Z565P" H 8800 6200 60  0001 C CNN
+F 3 "" H 8800 6200 60  0000 C CNN
+	1    8800 6200
+	1    0    0    -1
+$EndComp
 $EndSCHEMATC

Commit message: initial layout
Other:
- moved on the sheet: C107
Changed lines of the file:
@@
 L C C107
 U 1 1 54888B9A
-P 2750 1900
-F 0 "C107" H 2775 1950 30  0000 L CNN
-F 1 "0.1uF" H 2775 1850 30  0000 L CNN
-F 2 "kicadlib:CAPC2012X100N" H 2750 1900 60  0001 C CNN
-F 3 "" H 2750 1900 60  0000 C CNN
-	1    2750 1900
+P 2650 2400
+F 0 "C107" H 2675 2450 30  0000 L CNN
+F 1 "0.1uF" H 2675 2350 30  0000 L CNN
+F 2 "kicadlib:CAPC2012X100N" H 2650 2400 60  0001 C CNN
+F 3 "" H 2650 2400 60  0000 C CNN
+	1    2650 2400
 	1    0    0    -1
 $EndComp
@@
 Wire Wire Line
 	2550 1750 2550 1800
-Wire Wire Line
-	1950 1750 2750 1750
 Connection ~ 1950 1750
 Wire Wire Line
@@
 	1950 2000 1950 2100
 Wire Wire Line
-	1950 2050 2750 2050
-Wire Wire Line
 	2550 2050 2550 2000
 Connection ~ 1950 2050
@@
 	2150 2000 2150 2050
 Connection ~ 2150 2050
-Wire Wire Line
-	2750 1750 2750 1800
 Connection ~ 2550 1750
-Wire Wire Line
-	2750 2050 2750 2000
 Connection ~ 2550 2050
 Wire Wire Line
@@
 	1    0    0    -1
 $EndComp
+$Comp
+L GNDPWR #PWR013
+U 1 1 54BC0F12
+P 2650 2600
+F 0 "#PWR013" H 2650 2650 40  0001 C CNN
+F 1 "GNDPWR" H 2650 2520 40  0001 C CNN
+F 2 "" H 2650 2600 60  0000 C CNN
+F 3 "" H 2650 2600 60  0000 C CNN
+	1    2650 2600
+	1    0    0    -1
+$EndComp
+Wire Wire Line
+	2650 2200 2650 2300
+Connection ~ 2650 2200
+Wire Wire Line
+	2650 2500 2650 2600
+Wire Wire Line
+	2550 1750 1950 1750
+Wire Wire Line
+	1950 2050 2550 2050
 $EndSCHEMATC
