File: hardware/stm32-wifi-door-bell.sch (KiCad schematic (older format))
At the start: 25 parts, among them J101 USB, M101 Mounting Hole, M102 Mounting Hole, M103 Mounting Hole, M104 Mounting Hole, P101 SWD, P102 FTDI-PLUG, U101 STM32F072CBT6, X101 32.768kHz, X102 8MHz

Commit message: clean up pcb
Parts:
- added S101: RESET, kicadlib:CKCOMP-PTS525SM10SMTR, symbol SPST-4PIN
Connections:
- wire segments 103 -> 110
Changed lines of the file:
@@
 Text Label 1450 3400 0    60   ~ 0
 USBDPPU
-Text Label 5900 3100 2    60   ~ 0
+Text Label 5900 2000 2    60   ~ 0
 USBDPPU
 $Comp
@@
 Text Label 5900 2500 2    60   ~ 0
 SPI1MOSI
+Text Label 5900 3400 2    60   ~ 0
+CC3000CS
 Text Label 5900 3300 2    60   ~ 0
-CC3000CS
-Text Label 5900 3400 2    60   ~ 0
 CC3000IRQ
 Text Label 5900 3500 2    60   ~ 0
@@
 Text Label 5900 3700 2    60   ~ 0
 BTNBACK
-NoConn ~ 5400 2000
 NoConn ~ 5400 2100
 NoConn ~ 5400 3800
@@
 	5900 2800 5400 2800
 Wire Wire Line
-	5900 3100 5400 3100
-Wire Wire Line
 	2000 7200 2100 7200
 Wire Wire Line
@@
 	1950 2050 2550 2050
 NoConn ~ 5400 4300
+Wire Wire Line
+	5900 2000 5400 2000
+NoConn ~ 5400 3100
+$Comp
+L SPST-4PIN S101
+U 1 1 54BFAC50
+P 2350 5050
+F 0 "S101" H 2300 5350 60  0000 C CNN
+F 1 "RESET" H 2350 4950 60  0000 C CNN
+F 2 "kicadlib:CKCOMP-PTS525SM10SMTR" H 2350 5050 60  0001 C CNN
+F 3 "" H 2350 5050 60  0000 C CNN
+	1    2350 5050
+	1    0    0    -1
+$EndComp
+$Comp
+L GNDPWR #PWR014
+U 1 1 54BFB87B
+P 2000 5200
+F 0 "#PWR014" H 2000 5250 40  0001 C CNN
+F 1 "GNDPWR" H 2000 5120 40  0001 C CNN
+F 2 "" H 2000 5200 60  0000 C CNN
+F 3 "" H 2000 5200 60  0000 C CNN
+	1    2000 5200
+	1    0    0    -1
+$EndComp
+Wire Wire Line
+	2850 4300 2850 5050
+Wire Wire Line
+	2850 5050 2600 5050
+Wire Wire Line
+	2600 4950 2650 4950
+Wire Wire Line
+	2650 4950 2650 5050
+Connection ~ 2650 5050
+Wire Wire Line
+	2100 4950 2000 4950
+Wire Wire Line
+	2000 4950 2000 5200
+Wire Wire Line
+	2100 5050 2000 5050
+Connection ~ 2000 5050
 $EndSCHEMATC

Commit message: v20150125
Parts:
- BT101: inventoryId (none) -> 289
- C101, C102, C103, C105, C107: inventoryId (none) -> 10
- C104, C106: inventoryId (none) -> 446
- C108, C109, C110, C111: inventoryId (none) -> 388
- J101: inventoryId (none) -> 274
- M101, M102, M103, M104, P101, P102: inventoryId (none) -> NA
- R101: inventoryId (none) -> 391
- R102, R103: inventoryId (none) -> 49
- S101: inventoryId (none) -> 275
- U101: inventoryId (none) -> 604
- X101: inventoryId (none) -> 280
- X102: inventoryId (none) -> 488
Changed lines of the file:
@@
 F 2 "kicadlib:QFP50P900X900X160-48N" H 4400 3400 60  0001 C CNN
 F 3 "" H 4400 3400 60  0000 C CNN
+F 4 "604" H 4400 3400 60  0001 C CNN "inventoryId"
 	1    4400 3400
 	1    0    0    -1
@@
 F 2 "kicadlib:HDRV6W66P254_1X6_1524X249X838P" H 3400 7200 60  0001 C CNN
 F 3 "" H 3400 7200 60  0000 C CNN
+F 4 "NA" H 3700 7300 60  0001 C CNN "inventoryId"
 	1    3700 7300
 	1    0    0    -1
@@
 F 2 "kicadlib:HDRV6W66P254_1X6_1524X249X838P" H 5600 7100 60  0001 C CNN
 F 3 "" H 5600 7100 60  0000 C CNN
+F 4 "NA" H 5600 7300 60  0001 C CNN "inventoryId"
 	1    5600 7300
 	1    0    0    -1
@@
 F 2 "kicadlib:SOJ550P370X240-4N" H 3350 2650 60  0001 C CNN
 F 3 "" H 3350 2650 60  0000 C CNN
+F 4 "280" H 3350 2650 60  0001 C CNN "inventoryId"
 	1    3350 2650
 	0    1    1    0
@@
 F 2 "kicadlib:XTAL8045X200N" H 3350 3350 60  0001 C CNN
 F 3 "" H 3350 3350 60  0000 C CNN
+F 4 "488" H 3350 3350 60  0001 C CNN "inventoryId"
 	1    3350 3350
 	0    1    1    0
@@
 F 2 "kicadlib:CAPC2012X100N" H 3150 3600 60  0001 C CNN
 F 3 "" H 3150 3600 60  0000 C CNN
+F 4 "388" H 3150 3600 60  0001 C CNN "inventoryId"
 	1    3150 3600
 	0    1    1    0
@@
 F 2 "kicadlib:CAPC2012X100N" H 3150 3100 60  0001 C CNN
 F 3 "" H 3150 3100 60  0000 C CNN
+F 4 "388" H 3150 3100 60  0001 C CNN "inventoryId"
 	1    3150 3100
 	0    1    1    0
@@
 F 2 "kicadlib:CAPC2012X100N" H 3150 2900 60  0001 C CNN
 F 3 "" H 3150 2900 60  0000 C CNN
+F 4 "388" H 3150 2900 60  0001 C CNN "inventoryId"
 	1    3150 2900
 	0    1    1    0
@@
 F 2 "kicadlib:CAPC2012X100N" H 3150 2400 60  0001 C CNN
 F 3 "" H 3150 2400 60  0000 C CNN
+F 4 "388" H 3150 2400 60  0001 C CNN "inventoryId"
 	1    3150 2400
 	0    1    1    0
@@
 F 2 "kicadlib:CAPC2012X100N" H 2650 4200 60  0001 C CNN
 F 3 "" H 2650 4200 60  0000 C CNN
+F 4 "446" H 2650 4200 60  0001 C CNN "inventoryId"
 	1    2650 4200
 	-1   0    0    1
@@
 F 2 "kicadlib:CAPC2012X100N" H 2450 4200 60  0001 C CNN
 F 3 "" H 2450 4200 60  0000 C CNN
+F 4 "446" H 2450 4200 60  0001 C CNN "inventoryId"
 	1    2450 4200
 	-1   0    0    1
@@
 F 2 "kicadlib:RESC2012X100N" H 2250 3900 60  0001 C CNN
 F 3 "" H 2250 3900 60  0000 C CNN
+F 4 "49" H 2250 3900 60  0001 C CNN "inventoryId"
 	1    2250 3900
 	0    1    1    0
@@
 F 2 "kicadlib:RESC2012X100N" H 2250 4000 60  0001 C CNN
 F 3 "" H 2250 4000 60  0000 C CNN
+F 4 "49" H 2250 4000 60  0001 C CNN "inventoryId"
 	1    2250 4000
 	0    1    1    0
@@
 F 2 "kicadlib:RESC2012X100N" H 2050 3600 60  0001 C CNN
 F 3 "" H 2050 3600 60  0000 C CNN
+F 4 "391" H 2050 3600 60  0001 C CNN "inventoryId"
 	1    2050 3600
 	1    0    0    -1
@@
 F 2 "kicadlib:JST_UB-MC5BR3-SD204-4S-NMP" H 1750 7000 60  0001 C CNN
 F 3 "" H 1750 7000 60  0000 C CNN
+F 4 "274" H 1800 7000 60  0001 C CNN "inventoryId"
 	1    1800 7000
 	1    0    0    -1
@@
 F 2 "kicadlib:CAPC2012X100N" H 1950 1900 60  0001 C CNN
 F 3 "" H 1950 1900 60  0000 C CNN
+F 4 "10" H 1950 1900 60  0001 C CNN "inventoryId"
 	1    1950 1900
 	1    0    0    -1
@@
 F 2 "kicadlib:CAPC2012X100N" H 2150 1900 60  0001 C CNN
 F 3 "" H 2150 1900 60  0000 C CNN
+F 4 "10" H 2150 1900 60  0001 C CNN "inventoryId"
 	1    2150 1900
 	1    0    0    -1
@@
 F 2 "kicadlib:CAPC2012X100N" H 2350 1900 60  0001 C CNN
 F 3 "" H 2350 1900 60  0000 C CNN
+F 4 "10" H 2350 1900 60  0001 C CNN "inventoryId"
 	1    2350 1900
 	1    0    0    -1
@@
 F 2 "kicadlib:CAPC2012X100N" H 2550 1900 60  0001 C CNN
 F 3 "" H 2550 1900 60  0000 C CNN
+F 4 "10" H 2550 1900 60  0001 C CNN "inventoryId"
 	1    2550 1900
 	1    0    0    -1
@@
 F 2 "kicadlib:CAPC2012X100N" H 2650 2400 60  0001 C CNN
 F 3 "" H 2650 2400 60  0000 C CNN
+F 4 "10" H 2650 2400 60  0001 C CNN "inventoryId"
 	1    2650 2400
 	1    0    0    -1
@@
 F 2 "kicadlib:KEYSTONE-3000" H 2350 2700 60  0001 C CNN
 F 3 "" H 2350 2700 60  0000 C CNN
+F 4 "289" H 2350 2700 60  0001 C CNN "inventoryId"
 	1    2350 2700
 	0    1    1    0
@@
 F 2 "kicadlib:MTGNP565H328Z565P" H 8800 5900 60  0001 C CNN
 F 3 "" H 8800 5900 60  0000 C CNN
+F 4 "NA" H 8800 5900 60  0001 C CNN "inventoryId"
 	1    8800 5900
 	1    0    0    -1
@@
 F 2 "kicadlib:MTGNP565H328Z565P" H 8800 6000 60  0001 C CNN
 F 3 "" H 8800 6000 60  0000 C CNN
+F 4 "NA" H 8800 6000 60  0001 C CNN "inventoryId"
 	1    8800 6000
 	1    0    0    -1
@@
 F 2 "kicadlib:MTGNP565H328Z565P" H 8800 6100 60  0001 C CNN
 F 3 "" H 8800 6100 60  0000 C CNN
+F 4 "NA" H 8800 6100 60  0001 C CNN "inventoryId"
 	1    8800 6100
 	1    0    0    -1
@@
 F 2 "kicadlib:MTGNP565H328Z565P" H 8800 6200 60  0001 C CNN
 F 3 "" H 8800 6200 60  0000 C CNN
+F 4 "NA" H 8800 6200 60  0001 C CNN "inventoryId"
 	1    8800 6200
 	1    0    0    -1
@@
 F 2 "kicadlib:CKCOMP-PTS525SM10SMTR" H 2350 5050 60  0001 C CNN
 F 3 "" H 2350 5050 60  0000 C CNN
+F 4 "275" H 2350 5050 60  0001 C CNN "inventoryId"
 	1    2350 5050
 	1    0    0    -1
