File: hardware/stm32-wifi-door-bell-power.sch (KiCad schematic (older format))
At the start: 11 parts, among them U6 MC34063A

Commit message: reannotate schematic
Parts:
- renumbered C16 to C301, C20 to C302, C22 to C303, D2 to D301, D5 to D302, L1 to L301, L4 to L302, R8 to R301, R14 to R302, R16 to R303, U6 to U301
Changed lines of the file:
@@
 $EndDescr
 $Comp
-L Vcc #PWR39
+L Vcc #PWR301
 U 1 1 54B1D935
 P 4850 3350
-F 0 "#PWR39" H 4850 3440 20  0001 C CNN
+F 0 "#PWR301" H 4850 3440 20  0001 C CNN
 F 1 "Vcc" H 4850 3440 30  0000 C CNN
 F 2 "" H 4850 3350 60  0000 C CNN
@@
 	7150 3750 6550 3750
 $Comp
-L INDUCTOR L1
+L INDUCTOR L301
 U 1 1 54B1D958
 P 6900 3250
-F 0 "L1" H 6900 3200 30  0000 C CNN
+F 0 "L301" H 6900 3200 30  0000 C CNN
 F 1 ">70uH" H 6900 3300 30  0000 C CNN
 F 2 "" H 6900 3250 60  0000 C CNN
@@
 	6550 3250 6750 3250
 $Comp
-L GNDPWR #PWR43
+L GNDPWR #PWR305
 U 1 1 54B1D989
 P 6650 3600
-F 0 "#PWR43" H 6650 3650 40  0001 C CNN
+F 0 "#PWR305" H 6650 3650 40  0001 C CNN
 F 1 "GNDPWR" H 6650 3520 40  0001 C CNN
 F 2 "" H 6650 3600 60  0000 C CNN
@@
 	4850 3850 4850 3950
 $Comp
-L Vcc #PWR40
+L Vcc #PWR302
 U 1 1 54B1D9CE
 P 4850 3350
-F 0 "#PWR40" H 4850 3440 20  0001 C CNN
+F 0 "#PWR302" H 4850 3440 20  0001 C CNN
 F 1 "Vcc" H 4850 3440 30  0000 C CNN
 F 2 "" H 4850 3350 60  0000 C CNN
@@
 $EndComp
 $Comp
-L +3.3V #PWR47
+L +3.3V #PWR309
 U 1 1 54B1D9D7
 P 7450 3150
-F 0 "#PWR47" H 7450 3240 20  0001 C CNN
+F 0 "#PWR309" H 7450 3240 20  0001 C CNN
 F 1 "+3.3V" H 7450 3240 30  0000 C CNN
 F 2 "" H 7450 3150 60  0000 C CNN
@@
 $EndComp
 $Comp
-L GNDPWR #PWR48
+L GNDPWR #PWR310
 U 1 1 54B1D9E0
 P 7450 4250
-F 0 "#PWR48" H 7450 4300 40  0001 C CNN
+F 0 "#PWR310" H 7450 4300 40  0001 C CNN
 F 1 "GNDPWR" H 7450 4170 40  0001 C CNN
 F 2 "" H 7450 4250 60  0000 C CNN
@@
 $EndComp
 $Comp
-L CP C22
+L CP C303
 U 1 1 54B1D9E6
 P 7450 3500
-F 0 "C22" H 7475 3550 30  0000 L CNN
+F 0 "C303" H 7475 3550 30  0000 L CNN
 F 1 "100uF" H 7475 3450 30  0000 L CNN
 F 2 "" H 7450 3500 60  0000 C CNN
@@
 $EndComp
 $Comp
-L INDUCTOR L4
+L INDUCTOR L302
 U 1 1 54B1D9F1
 P 6900 3250
-F 0 "L4" H 6900 3200 30  0000 C CNN
+F 0 "L302" H 6900 3200 30  0000 C CNN
 F 1 ">70uH" H 6900 3300 30  0000 C CNN
 F 2 "" H 6900 3250 60  0000 C CNN
@@
 $EndComp
 $Comp
-L GNDPWR #PWR46
+L GNDPWR #PWR308
 U 1 1 54B1D9F9
 P 7150 4250
-F 0 "#PWR46" H 7150 4300 40  0001 C CNN
+F 0 "#PWR308" H 7150 4300 40  0001 C CNN
 F 1 "GNDPWR" H 7150 4170 40  0001 C CNN
 F 2 "" H 7150 4250 60  0000 C CNN
@@
 $EndComp
 $Comp
-L R R14
+L R R302
 U 1 1 54B1DA01
 P 7150 3500
-F 0 "R14" V 7095 3500 30  0000 C CNN
+F 0 "R302" V 7095 3500 30  0000 C CNN
 F 1 "18K" V 7050 3500 30  0000 C CNN
 F 2 "kicadlib:RESC2012X100N" H 7150 3500 60  0001 C CNN
@@
 $EndComp
 $Comp
-L R R16
+L R R303
 U 1 1 54B1DA08
 P 7150 4050
-F 0 "R16" V 7095 4050 30  0000 C CNN
+F 0 "R303" V 7095 4050 30  0000 C CNN
 F 1 "11K" V 7050 4050 30  0000 C CNN
 F 2 "kicadlib:RESC2012X100N" H 7150 4050 60  0001 C CNN
@@
 $EndComp
 $Comp
-L GNDPWR #PWR45
+L GNDPWR #PWR307
 U 1 1 54B1DA10
 P 6650 4250
-F 0 "#PWR45" H 6650 4300 40  0001 C CNN
+F 0 "#PWR307" H 6650 4300 40  0001 C CNN
 F 1 "GNDPWR" H 6650 4170 40  0001 C CNN
 F 2 "" H 6650 4250 60  0000 C CNN
@@
 $EndComp
 $Comp
-L C C20
+L C C302
 U 1 1 54B1DA18
 P 6650 4050
-F 0 "C20" H 6675 4100 30  0000 L CNN
+F 0 "C302" H 6675 4100 30  0000 L CNN
 F 1 "240pF" H 6675 4000 30  0000 L CNN
 F 2 "kicadlib:CAPC2012X100N" H 6650 4050 60  0001 C CNN
@@
 $EndComp
 $Comp
-L GNDPWR #PWR44
+L GNDPWR #PWR306
 U 1 1 54B1DA22
 P 6650 3600
-F 0 "#PWR44" H 6650 3650 40  0001 C CNN
+F 0 "#PWR306" H 6650 3650 40  0001 C CNN
 F 1 "GNDPWR" H 6650 3520 40  0001 C CNN
 F 2 "" H 6650 3600 60  0000 C CNN
@@
 $EndComp
 $Comp
-L DIODESCH D5
+L DIODESCH D302
 U 1 1 54B1DA28
 P 6650 3450
-F 0 "D5" H 6650 3550 40  0000 C CNN
+F 0 "D302" H 6650 3550 40  0000 C CNN
 F 1 ">3.3V" H 6650 3350 40  0000 C CNN
 F 2 "" H 6650 3450 60  0000 C CNN
@@
 $EndComp
 $Comp
-L R R8
+L R R301
 U 1 1 54B1DA39
 P 5150 3350
-F 0 "R8" V 5095 3350 30  0000 C CNN
+F 0 "R301" V 5095 3350 30  0000 C CNN
 F 1 "0.3R" V 5050 3350 30  0000 C CNN
 F 2 "kicadlib:RESC2012X100N" H 5150 3350 60  0001 C CNN
@@
 $EndComp
 $Comp
-L GNDPWR #PWR42
+L GNDPWR #PWR304
 U 1 1 54B1DA43
 P 5250 3950
-F 0 "#PWR42" H 5250 4000 40  0001 C CNN
+F 0 "#PWR304" H 5250 4000 40  0001 C CNN
 F 1 "GNDPWR" H 5250 3870 40  0001 C CNN
 F 2 "" H 5250 3950 60  0000 C CNN
@@
 $EndComp
 $Comp
-L MC34063A U6
+L MC34063A U301
 U 1 1 54B1DA49
 P 5850 3450
-F 0 "U6" H 5550 4000 60  0000 L CNN
+F 0 "U301" H 5550 4000 60  0000 L CNN
 F 1 "MC34063A" H 5550 2900 60  0000 L CNN
 F 2 "" H 5850 2950 60  0000 C CNN
@@
 $EndComp
 $Comp
-L GNDPWR #PWR41
+L GNDPWR #PWR303
 U 1 1 54B1DA53
 P 4850 3950
-F 0 "#PWR41" H 4850 4000 40  0001 C CNN
+F 0 "#PWR303" H 4850 4000 40  0001 C CNN
 F 1 "GNDPWR" H 4850 3870 40  0001 C CNN
 F 2 "" H 4850 3950 60  0000 C CNN
@@
 $EndComp
 $Comp
-L CP C16
+L CP C301
 U 1 1 54B1DA59
 P 4850 3750
-F 0 "C16" H 4875 3800 30  0000 L CNN
+F 0 "C301" H 4875 3800 30  0000 L CNN
 F 1 "1000uF" H 4875 3700 30  0000 L CNN
 F 2 "" H 4850 3750 60  0000 C CNN
@@
 $EndComp
 $Comp
-L DIODESCH D2
+L DIODESCH D301
 U 1 1 54B1DA60
 P 4550 3550
-F 0 "D2" H 4550 3650 40  0000 C CNN
+F 0 "D301" H 4550 3650 40  0000 C CNN
 F 1 ">20V 500mA" H 4550 3450 40  0000 C CNN
 F 2 "" H 4550 3550 60  0000 C CNN
@@
 FRONTIN
 $Comp
-L PWR_FLAG #FLG1
+L PWR_FLAG #FLG301
 U 1 1 54B179C7
 P 4650 3350
-F 0 "#FLG1" H 4650 3445 30  0001 C CNN
+F 0 "#FLG301" H 4650 3445 30  0001 C CNN
 F 1 "PWR_FLAG" H 4650 3440 30  0000 C CNN
 F 2 "" H 4650 3350 60  0000 C CNN
@@
 Connection ~ 4850 3400
 $Comp
-L PWR_FLAG #FLG2
+L PWR_FLAG #FLG302
 U 1 1 54B17E6C
 P 7700 3150
-F 0 "#FLG2" H 7700 3245 30  0001 C CNN
+F 0 "#FLG302" H 7700 3245 30  0001 C CNN
 F 1 "PWR_FLAG" H 7700 3240 30  0000 C CNN
 F 2 "" H 7700 3150 60  0000 C CNN

Commit message: more schematics
Parts:
- added D303: >20V 500mA, kicadlib:DIOM5226X220N, symbol DIODESCH
- added D304, D305: LED, kicadlib:LEDC3216X100N, symbol LED
- added R304, R305: 1K, kicadlib:RESC2012X100N, symbol R
- C301: value 1000uF -> 2200uF
- D301, D302: footprint (none) -> kicadlib:DIOM5226X220N
Connections:
- net labels added: BACKIN
- wire segments 29 -> 37
Other:
- moved on the sheet: C302, L301, L302, R301, R302, R303

Commit message: initial layout
Parts:
- removed L302: >70uH, symbol INDUCTOR
- C301: value 2200uF -> 2200uF >16V; footprint (none) -> kicadlib:CAPPRD750W80D1600H2500P
- C303: footprint (none) -> kicadlib:CAPAE660X790N
- L301: footprint (none) -> kicadlib:IND_ASPI-8040S-680M-T; MfgPartNumber (none) -> ASPI-8040S-101M-T
- U301: footprint (none) -> kicadlib:SOIC127P600X175-8N
Changed lines of the file:
@@
 $EndDescr
 $Comp
-L Vcc #PWR033
+L Vcc #PWR034
 U 1 1 54B1D935
 P 4300 3300
-F 0 "#PWR033" H 4300 3390 20  0001 C CNN
+F 0 "#PWR034" H 4300 3390 20  0001 C CNN
 F 1 "Vcc" H 4300 3390 30  0000 C CNN
 F 2 "" H 4300 3300 60  0000 C CNN
@@
 F 0 "L301" H 6850 3150 30  0000 C CNN
 F 1 ">70uH" H 6850 3250 30  0000 C CNN
-F 2 "" H 6850 3200 60  0001 C CNN
+F 2 "kicadlib:IND_ASPI-8040S-680M-T" H 6850 3200 60  0001 C CNN
 F 3 "" H 6850 3200 60  0000 C CNN
+F 4 "ASPI-8040S-101M-T" H 6850 3200 60  0001 C CNN "MfgPartNumber"
 	1    6850 3200
 	1    0    0    -1
@@
 	6500 3200 6700 3200
 $Comp
-L GNDPWR #PWR034
+L GNDPWR #PWR035
 U 1 1 54B1D989
 P 6600 3550
-F 0 "#PWR034" H 6600 3600 40  0001 C CNN
+F 0 "#PWR035" H 6600 3600 40  0001 C CNN
 F 1 "GNDPWR" H 6600 3470 40  0001 C CNN
 F 2 "" H 6600 3550 60  0000 C CNN
@@
 	4300 3800 4300 3900
 $Comp
-L Vcc #PWR035
+L Vcc #PWR036
 U 1 1 54B1D9CE
 P 4300 3300
-F 0 "#PWR035" H 4300 3390 20  0001 C CNN
+F 0 "#PWR036" H 4300 3390 20  0001 C CNN
 F 1 "Vcc" H 4300 3390 30  0000 C CNN
 F 2 "" H 4300 3300 60  0000 C CNN
@@
 $EndComp
 $Comp
-L +3.3V #PWR036
+L +3.3V #PWR037
 U 1 1 54B1D9D7
 P 7400 3100
-F 0 "#PWR036" H 7400 3190 20  0001 C CNN
+F 0 "#PWR037" H 7400 3190 20  0001 C CNN
 F 1 "+3.3V" H 7400 3190 30  0000 C CNN
 F 2 "" H 7400 3100 60  0000 C CNN
@@
 $EndComp
 $Comp
-L GNDPWR #PWR037
+L GNDPWR #PWR038
 U 1 1 54B1D9E0
 P 7400 4200
-F 0 "#PWR037" H 7400 4250 40  0001 C CNN
+F 0 "#PWR038" H 7400 4250 40  0001 C CNN
 F 1 "GNDPWR" H 7400 4120 40  0001 C CNN
 F 2 "" H 7400 4200 60  0000 C CNN
@@
 F 0 "C303" H 7425 3500 30  0000 L CNN
 F 1 "100uF" H 7425 3400 30  0000 L CNN
-F 2 "" H 7400 3450 60  0001 C CNN
+F 2 "kicadlib:CAPAE660X790N" H 7400 3450 60  0001 C CNN
 F 3 "" H 7400 3450 60  0000 C CNN
 	1    7400 3450
@@
 $EndComp
 $Comp
-L INDUCTOR L302
-U 1 1 54B1D9F1
-P 6850 3200
-F 0 "L302" H 6850 3150 30  0000 C CNN
-F 1 ">70uH" H 6850 3250 30  0000 C CNN
-F 2 "" H 6850 3200 60  0001 C CNN
-F 3 "" H 6850 3200 60  0000 C CNN
-	1    6850 3200
-	1    0    0    -1
-$EndComp
-$Comp
-L GNDPWR #PWR038
+L GNDPWR #PWR039
 U 1 1 54B1D9F9
 P 7100 4200
-F 0 "#PWR038" H 7100 4250 40  0001 C CNN
+F 0 "#PWR039" H 7100 4250 40  0001 C CNN
 F 1 "GNDPWR" H 7100 4120 40  0001 C CNN
 F 2 "" H 7100 4200 60  0000 C CNN
@@
 $EndComp
 $Comp
-L GNDPWR #PWR039
+L GNDPWR #PWR040
 U 1 1 54B1DA10
 P 6600 4200
-F 0 "#PWR039" H 6600 4250 40  0001 C CNN
+F 0 "#PWR040" H 6600 4250 40  0001 C CNN
 F 1 "GNDPWR" H 6600 4120 40  0001 C CNN
 F 2 "" H 6600 4200 60  0000 C CNN
@@
 $EndComp
 $Comp
-L GNDPWR #PWR040
+L GNDPWR #PWR041
 U 1 1 54B1DA22
 P 6600 3550
-F 0 "#PWR040" H 6600 3600 40  0001 C CNN
+F 0 "#PWR041" H 6600 3600 40  0001 C CNN
 F 1 "GNDPWR" H 6600 3470 40  0001 C CNN
 F 2 "" H 6600 3550 60  0000 C CNN
@@
 $EndComp
 $Comp
-L GNDPWR #PWR041
+L GNDPWR #PWR042
 U 1 1 54B1DA43
 P 5200 3900
-F 0 "#PWR041" H 5200 3950 40  0001 C CNN
+F 0 "#PWR042" H 5200 3950 40  0001 C CNN
 F 1 "GNDPWR" H 5200 3820 40  0001 C CNN
 F 2 "" H 5200 3900 60  0000 C CNN
@@
 F 0 "U301" H 5500 3950 60  0000 L CNN
 F 1 "MC34063A" H 5500 2850 60  0000 L CNN
-F 2 "" H 5800 2900 60  0001 C CNN
+F 2 "kicadlib:SOIC127P600X175-8N" H 5800 2900 60  0001 C CNN
 F 3 "" H 5800 2900 60  0000 C CNN
 	1    5800 3400
@@
 $EndComp
 $Comp
-L GNDPWR #PWR042
+L GNDPWR #PWR043
 U 1 1 54B1DA53
 P 4300 3900
-F 0 "#PWR042" H 4300 3950 40  0001 C CNN
+F 0 "#PWR043" H 4300 3950 40  0001 C CNN
 F 1 "GNDPWR" H 4300 3820 40  0001 C CNN
 F 2 "" H 4300 3900 60  0000 C CNN
@@
 P 4300 3700
 F 0 "C301" H 4325 3750 30  0000 L CNN
-F 1 "2200uF" H 4325 3650 30  0000 L CNN
-F 2 "" H 4300 3700 60  0001 C CNN
+F 1 "2200uF >16V" H 4325 3650 30  0000 L CNN
+F 2 "kicadlib:CAPPRD750W80D1600H2500P" H 4300 3700 60  0001 C CNN
 F 3 "" H 4300 3700 60  0000 C CNN
 	1    4300 3700
@@
 FRONTIN
 $Comp
-L PWR_FLAG #FLG043
+L PWR_FLAG #FLG044
 U 1 1 54B179C7
 P 4100 3300
-F 0 "#FLG043" H 4100 3395 30  0001 C CNN
+F 0 "#FLG044" H 4100 3395 30  0001 C CNN
 F 1 "PWR_FLAG" H 4100 3390 30  0000 C CNN
 F 2 "" H 4100 3300 60  0000 C CNN
@@
 Connection ~ 4300 3350
 $Comp
-L PWR_FLAG #FLG044
+L PWR_FLAG #FLG045
 U 1 1 54B17E6C
 P 7650 3100
-F 0 "#FLG044" H 7650 3195 30  0001 C CNN
+F 0 "#FLG045" H 7650 3195 30  0001 C CNN
 F 1 "PWR_FLAG" H 7650 3190 30  0000 C CNN
 F 2 "" H 7650 3100 60  0000 C CNN
@@
 $EndComp
 $Comp
-L GNDPWR #PWR045
+L GNDPWR #PWR046
 U 1 1 54B5D31F
 P 4700 4200
-F 0 "#PWR045" H 4700 4250 40  0001 C CNN
+F 0 "#PWR046" H 4700 4250 40  0001 C CNN
 F 1 "GNDPWR" H 4700 4120 40  0001 C CNN
 F 2 "" H 4700 4200 60  0000 C CNN
@@
 $EndComp
 $Comp
-L GNDPWR #PWR046
+L GNDPWR #PWR047
 U 1 1 54B5D72C
 P 4000 6000
-F 0 "#PWR046" H 4000 6050 40  0001 C CNN
+F 0 "#PWR047" H 4000 6050 40  0001 C CNN
 F 1 "GNDPWR" H 4000 5920 40  0001 C CNN
 F 2 "" H 4000 6000 60  0000 C CNN

Commit message: clean up pcb
Parts:
- added P301: PWR, kicadlib:HDRV2W66P254_1X2_508X249X838P, symbol P02
Connections:
- wire segments 37 -> 41
Changed lines of the file:
@@
 $EndDescr
 $Comp
-L Vcc #PWR034
+L Vcc #PWR035
 U 1 1 54B1D935
 P 4300 3300
-F 0 "#PWR034" H 4300 3390 20  0001 C CNN
+F 0 "#PWR035" H 4300 3390 20  0001 C CNN
 F 1 "Vcc" H 4300 3390 30  0000 C CNN
 F 2 "" H 4300 3300 60  0000 C CNN
@@
 	6500 3200 6700 3200
 $Comp
-L GNDPWR #PWR035
+L GNDPWR #PWR036
 U 1 1 54B1D989
 P 6600 3550
-F 0 "#PWR035" H 6600 3600 40  0001 C CNN
+F 0 "#PWR036" H 6600 3600 40  0001 C CNN
 F 1 "GNDPWR" H 6600 3470 40  0001 C CNN
 F 2 "" H 6600 3550 60  0000 C CNN
@@
 	4300 3800 4300 3900
 $Comp
-L Vcc #PWR036
+L Vcc #PWR037
 U 1 1 54B1D9CE
 P 4300 3300
-F 0 "#PWR036" H 4300 3390 20  0001 C CNN
+F 0 "#PWR037" H 4300 3390 20  0001 C CNN
 F 1 "Vcc" H 4300 3390 30  0000 C CNN
 F 2 "" H 4300 3300 60  0000 C CNN
@@
 $EndComp
 $Comp
-L +3.3V #PWR037
+L +3.3V #PWR038
 U 1 1 54B1D9D7
 P 7400 3100
-F 0 "#PWR037" H 7400 3190 20  0001 C CNN
+F 0 "#PWR038" H 7400 3190 20  0001 C CNN
 F 1 "+3.3V" H 7400 3190 30  0000 C CNN
 F 2 "" H 7400 3100 60  0000 C CNN
@@
 $EndComp
 $Comp
-L GNDPWR #PWR038
+L GNDPWR #PWR039
 U 1 1 54B1D9E0
 P 7400 4200
-F 0 "#PWR038" H 7400 4250 40  0001 C CNN
+F 0 "#PWR039" H 7400 4250 40  0001 C CNN
 F 1 "GNDPWR" H 7400 4120 40  0001 C CNN
 F 2 "" H 7400 4200 60  0000 C CNN
@@
 $EndComp
 $Comp
-L GNDPWR #PWR039
+L GNDPWR #PWR040
 U 1 1 54B1D9F9
 P 7100 4200
-F 0 "#PWR039" H 7100 4250 40  0001 C CNN
+F 0 "#PWR040" H 7100 4250 40  0001 C CNN
 F 1 "GNDPWR" H 7100 4120 40  0001 C CNN
 F 2 "" H 7100 4200 60  0000 C CNN
@@
 $EndComp
 $Comp
-L GNDPWR #PWR040
+L GNDPWR #PWR041
 U 1 1 54B1DA10
 P 6600 4200
-F 0 "#PWR040" H 6600 4250 40  0001 C CNN
+F 0 "#PWR041" H 6600 4250 40  0001 C CNN
 F 1 "GNDPWR" H 6600 4120 40  0001 C CNN
 F 2 "" H 6600 4200 60  0000 C CNN
@@
 $EndComp
 $Comp
-L GNDPWR #PWR041
+L GNDPWR #PWR042
 U 1 1 54B1DA22
 P 6600 3550
-F 0 "#PWR041" H 6600 3600 40  0001 C CNN
+F 0 "#PWR042" H 6600 3600 40  0001 C CNN
 F 1 "GNDPWR" H 6600 3470 40  0001 C CNN
 F 2 "" H 6600 3550 60  0000 C CNN
@@
 $EndComp
 $Comp
-L GNDPWR #PWR042
+L GNDPWR #PWR043
 U 1 1 54B1DA43
 P 5200 3900
-F 0 "#PWR042" H 5200 3950 40  0001 C CNN
+F 0 "#PWR043" H 5200 3950 40  0001 C CNN
 F 1 "GNDPWR" H 5200 3820 40  0001 C CNN
 F 2 "" H 5200 3900 60  0000 C CNN
@@
 $EndComp
 $Comp
-L GNDPWR #PWR043
+L GNDPWR #PWR044
 U 1 1 54B1DA53
 P 4300 3900
-F 0 "#PWR043" H 4300 3950 40  0001 C CNN
+F 0 "#PWR044" H 4300 3950 40  0001 C CNN
 F 1 "GNDPWR" H 4300 3820 40  0001 C CNN
 F 2 "" H 4300 3900 60  0000 C CNN
@@
 FRONTIN
 $Comp
-L PWR_FLAG #FLG044
+L PWR_FLAG #FLG045
 U 1 1 54B179C7
 P 4100 3300
-F 0 "#FLG044" H 4100 3395 30  0001 C CNN
+F 0 "#FLG045" H 4100 3395 30  0001 C CNN
 F 1 "PWR_FLAG" H 4100 3390 30  0000 C CNN
 F 2 "" H 4100 3300 60  0000 C CNN
@@
 Connection ~ 4300 3350
 $Comp
-L PWR_FLAG #FLG045
+L PWR_FLAG #FLG046
 U 1 1 54B17E6C
 P 7650 3100
-F 0 "#FLG045" H 7650 3195 30  0001 C CNN
+F 0 "#FLG046" H 7650 3195 30  0001 C CNN
 F 1 "PWR_FLAG" H 7650 3190 30  0000 C CNN
 F 2 "" H 7650 3100 60  0000 C CNN
@@
 $EndComp
 $Comp
-L GNDPWR #PWR046
+L GNDPWR #PWR047
 U 1 1 54B5D31F
 P 4700 4200
-F 0 "#PWR046" H 4700 4250 40  0001 C CNN
+F 0 "#PWR047" H 4700 4250 40  0001 C CNN
 F 1 "GNDPWR" H 4700 4120 40  0001 C CNN
 F 2 "" H 4700 4200 60  0000 C CNN
@@
 $EndComp
 $Comp
-L GNDPWR #PWR047
+L GNDPWR #PWR048
 U 1 1 54B5D72C
 P 4000 6000
-F 0 "#PWR047" H 4000 6050 40  0001 C CNN
+F 0 "#PWR048" H 4000 6050 40  0001 C CNN
 F 1 "GNDPWR" H 4000 5920 40  0001 C CNN
 F 2 "" H 4000 6000 60  0000 C CNN
@@
 Wire Wire Line
 	4000 5900 4000 6000
+$Comp
+L P02 P301
+U 1 1 54BC50D9
+P 6000 5100
+F 0 "P301" H 6050 5150 60  0000 C CNN
+F 1 "PWR" H 6000 4750 60  0000 L CNN
+F 2 "kicadlib:HDRV2W66P254_1X2_508X249X838P" H 6000 5100 60  0001 C CNN
+F 3 "" H 6000 5100 60  0000 C CNN
+	1    6000 5100
+	1    0    0    -1
+$EndComp
+$Comp
+L +3.3V #PWR049
+U 1 1 54BC522E
+P 5700 5100
+F 0 "#PWR049" H 5700 5190 20  0001 C CNN
+F 1 "+3.3V" H 5700 5190 30  0000 C CNN
+F 2 "" H 5700 5100 60  0000 C CNN
+F 3 "" H 5700 5100 60  0000 C CNN
+	1    5700 5100
+	1    0    0    -1
+$EndComp
+$Comp
+L GNDPWR #PWR050
+U 1 1 54BC526B
+P 5700 5400
+F 0 "#PWR050" H 5700 5450 40  0001 C CNN
+F 1 "GNDPWR" H 5700 5320 40  0001 C CNN
+F 2 "" H 5700 5400 60  0000 C CNN
+F 3 "" H 5700 5400 60  0000 C CNN
+	1    5700 5400
+	1    0    0    -1
+$EndComp
+Wire Wire Line
+	5800 5200 5700 5200
+Wire Wire Line
+	5700 5200 5700 5100
+Wire Wire Line
+	5800 5300 5700 5300
+Wire Wire Line
+	5700 5300 5700 5400
 $EndSCHEMATC

Commit message: v20150125
Parts:
- C301: inventoryId (none) -> 601
- C302: inventoryId (none) -> 608
- C303: inventoryId (none) -> 464
- D301, D302, D303: inventoryId (none) -> 273
- D304, D305: inventoryId (none) -> 177
- L301: inventoryId (none) -> 600
- P301: inventoryId (none) -> NA
- R301: inventoryId (none) -> 609
- R302: value 18K -> 16.2K; inventoryId (none) -> 610
- R303: value 11K -> 10K; inventoryId (none) -> 299
- R304, R305: inventoryId (none) -> 454
- U301: inventoryId (none) -> 272
Other:
- note added: "Vout=1.25(1+R302/R303)"
Changed lines of the file:
@@
 F 3 "" H 6850 3200 60  0000 C CNN
 F 4 "ASPI-8040S-101M-T" H 6850 3200 60  0001 C CNN "MfgPartNumber"
+F 5 "600" H 6850 3200 60  0001 C CNN "inventoryId"
 	1    6850 3200
 	1    0    0    -1
@@
 F 2 "kicadlib:CAPAE660X790N" H 7400 3450 60  0001 C CNN
 F 3 "" H 7400 3450 60  0000 C CNN
+F 4 "464" H 7400 3450 60  0001 C CNN "inventoryId"
 	1    7400 3450
 	1    0    0    -1
@@
 P 7100 3450
 F 0 "R302" V 7045 3450 30  0000 C CNN
-F 1 "18K" V 7000 3450 30  0000 C CNN
+F 1 "16.2K" V 7000 3450 30  0000 C CNN
 F 2 "kicadlib:RESC2012X100N" H 7100 3450 60  0001 C CNN
 F 3 "" H 7100 3450 60  0000 C CNN
+F 4 "610" H 7100 3450 60  0001 C CNN "inventoryId"
 	1    7100 3450
 	-1   0    0    1
@@
 P 7100 4000
 F 0 "R303" V 7045 4000 30  0000 C CNN
-F 1 "11K" V 7000 4000 30  0000 C CNN
+F 1 "10K" V 7000 4000 30  0000 C CNN
 F 2 "kicadlib:RESC2012X100N" H 7100 4000 60  0001 C CNN
 F 3 "" H 7100 4000 60  0000 C CNN
+F 4 "299" H 7100 4000 60  0001 C CNN "inventoryId"
 	1    7100 4000
 	-1   0    0    1
@@
 F 2 "kicadlib:CAPC2012X100N" H 6600 4000 60  0001 C CNN
 F 3 "" H 6600 4000 60  0000 C CNN
+F 4 "608" H 6600 4000 60  0001 C CNN "inventoryId"
 	1    6600 4000
 	1    0    0    -1
@@
 F 2 "kicadlib:DIOM5226X220N" H 6600 3400 60  0001 C CNN
 F 3 "" H 6600 3400 60  0000 C CNN
+F 4 "273" H 6600 3400 60  0001 C CNN "inventoryId"
 	1    6600 3400
 	0    -1   -1   0
@@
 F 2 "kicadlib:RESC2012X100N" H 5100 3300 60  0001 C CNN
 F 3 "" H 5100 3300 60  0000 C CNN
+F 4 "609" H 5100 3300 60  0001 C CNN "inventoryId"
 	1    5100 3300
 	-1   0    0    1
@@
 F 2 "kicadlib:SOIC127P600X175-8N" H 5800 2900 60  0001 C CNN
 F 3 "" H 5800 2900 60  0000 C CNN
+F 4 "272" H 5800 3400 60  0001 C CNN "inventoryId"
 	1    5800 3400
 	1    0    0    -1
@@
 F 2 "kicadlib:CAPPRD750W80D1600H2500P" H 4300 3700 60  0001 C CNN
 F 3 "" H 4300 3700 60  0000 C CNN
+F 4 "601" H 4300 3700 60  0001 C CNN "inventoryId"
 	1    4300 3700
 	1    0    0    -1
@@
 F 2 "kicadlib:DIOM5226X220N" H 4000 3500 60  0001 C CNN
 F 3 "" H 4000 3500 60  0000 C CNN
+F 4 "273" H 4000 3500 60  0001 C CNN "inventoryId"
 	1    4000 3500
 	1    0    0    -1
@@
 F 2 "kicadlib:LEDC3216X100N" H 4700 4000 60  0001 C CNN
 F 3 "" H 4700 4000 60  0000 C CNN
+F 4 "177" H 4700 4000 60  0001 C CNN "inventoryId"
 	1    4700 4000
 	0    1    1    0
@@
 F 2 "kicadlib:RESC2012X100N" H 4700 3700 60  0001 C CNN
 F 3 "" H 4700 3700 60  0000 C CNN
+F 4 "454" H 4700 3700 60  0001 C CNN "inventoryId"
 	1    4700 3700
 	-1   0    0    1
@@
 F 2 "kicadlib:RESC2012X100N" H 4000 5500 60  0001 C CNN
 F 3 "" H 4000 5500 60  0000 C CNN
+F 4 "454" H 4000 5500 60  0001 C CNN "inventoryId"
 	1    4000 5500
 	-1   0    0    1
@@
 F 2 "kicadlib:LEDC3216X100N" H 4000 5800 60  0001 C CNN
 F 3 "" H 4000 5800 60  0000 C CNN
+F 4 "177" H 4000 5800 60  0001 C CNN "inventoryId"
 	1    4000 5800
 	0    1    1    0
@@
 F 2 "kicadlib:DIOM5226X220N" H 3700 5200 60  0001 C CNN
 F 3 "" H 3700 5200 60  0000 C CNN
+F 4 "273" H 3700 5200 60  0001 C CNN "inventoryId"
 	1    3700 5200
 	1    0    0    -1
@@
 F 2 "kicadlib:HDRV2W66P254_1X2_508X249X838P" H 6000 5100 60  0001 C CNN
 F 3 "" H 6000 5100 60  0000 C CNN
+F 4 "NA" H 6000 5100 60  0001 C CNN "inventoryId"
 	1    6000 5100
 	1    0    0    -1
@@
 Wire Wire Line
 	5700 5300 5700 5400
+Text Notes 6650 4450 0    60   ~ 0
+Vout=1.25(1+R302/R303)
 $EndSCHEMATC
