File: hardware/stm32-wifi-door-bell-sdcard.sch (KiCad schematic (older format))
At the start: 3 parts

Commit message: reannotate schematic
Parts:
- gave numbers to parts that had none: 3
Changed lines of the file:
@@
 $EndDescr
 $Comp
-L MICROSD-AMPHENOL-114-00841-68 U?
+L MICROSD-AMPHENOL-114-00841-68 U501
 U 1 1 54B2F45D
 P 5950 3750
-F 0 "U?" H 5950 4450 60  0000 L CNN
+F 0 "U501" H 5950 4450 60  0000 L CNN
 F 1 "MICROSD-AMPHENOL-114-00841-68" H 5950 3450 60  0000 L CNN
 F 2 "" H 5950 3750 60  0000 C CNN
@@
 NoConn ~ 5750 3900
 $Comp
-L +3.3V #PWR?
+L +3.3V #PWR501
 U 1 1 54B2F466
 P 5650 2900
-F 0 "#PWR?" H 5650 2990 20  0001 C CNN
+F 0 "#PWR501" H 5650 2990 20  0001 C CNN
 F 1 "+3.3V" H 5650 2990 30  0000 C CNN
 F 2 "" H 5650 2900 60  0000 C CNN
@@
 $EndComp
 $Comp
-L GNDPWR #PWR?
+L GNDPWR #PWR502
 U 1 1 54B2F46C
 P 5650 4000
-F 0 "#PWR?" H 5650 4050 40  0001 C CNN
+F 0 "#PWR502" H 5650 4050 40  0001 C CNN
 F 1 "GNDPWR" H 5650 3920 40  0001 C CNN
 F 2 "" H 5650 4000 60  0000 C CNN
@@
 $EndComp
 $Comp
-L C C?
+L C C501
 U 1 1 54B2F476
 P 6750 3500
-F 0 "C?" H 6775 3550 30  0000 L CNN
+F 0 "C501" H 6775 3550 30  0000 L CNN
 F 1 "1uF" H 6775 3450 30  0000 L CNN
 F 2 "kicadlib:CAPC2012X100N" H 6750 3500 60  0001 C CNN
@@
 $EndComp
 $Comp
-L +3.3V #PWR?
+L +3.3V #PWR503
 U 1 1 54B2F47D
 P 6750 3300
-F 0 "#PWR?" H 6750 3390 20  0001 C CNN
+F 0 "#PWR503" H 6750 3390 20  0001 C CNN
 F 1 "+3.3V" H 6750 3390 30  0000 C CNN
 F 2 "" H 6750 3300 60  0000 C CNN
@@
 $EndComp
 $Comp
-L GNDPWR #PWR?
+L GNDPWR #PWR504
 U 1 1 54B2F483
 P 6750 3700
-F 0 "#PWR?" H 6750 3750 40  0001 C CNN
+F 0 "#PWR504" H 6750 3750 40  0001 C CNN
 F 1 "GNDPWR" H 6750 3620 40  0001 C CNN
 F 2 "" H 6750 3700 60  0000 C CNN
@@
 $EndComp
 $Comp
-L R R?
+L R R501
 U 1 1 54B2F489
 P 5500 3100
-F 0 "R?" V 5445 3100 30  0000 C CNN
+F 0 "R501" V 5445 3100 30  0000 C CNN
 F 1 "10K" V 5400 3100 30  0000 C CNN
 F 2 "kicadlib:RESC2012X100N" H 5500 3100 60  0001 C CNN

Commit message: more schematics
Changed lines of the file:
@@
 F 0 "U501" H 5950 4450 60  0000 L CNN
 F 1 "MICROSD-AMPHENOL-114-00841-68" H 5950 3450 60  0000 L CNN
-F 2 "" H 5950 3750 60  0000 C CNN
+F 2 "" H 5950 3750 60  0001 C CNN
 F 3 "" H 5950 3750 60  0000 C CNN
 	1    5950 3750
@@
 NoConn ~ 5750 3900
 $Comp
-L +3.3V #PWR501
+L +3.3V #PWR056
 U 1 1 54B2F466
 P 5650 2900
-F 0 "#PWR501" H 5650 2990 20  0001 C CNN
+F 0 "#PWR056" H 5650 2990 20  0001 C CNN
 F 1 "+3.3V" H 5650 2990 30  0000 C CNN
 F 2 "" H 5650 2900 60  0000 C CNN
@@
 $EndComp
 $Comp
-L GNDPWR #PWR502
+L GNDPWR #PWR057
 U 1 1 54B2F46C
 P 5650 4000
-F 0 "#PWR502" H 5650 4050 40  0001 C CNN
+F 0 "#PWR057" H 5650 4050 40  0001 C CNN
 F 1 "GNDPWR" H 5650 3920 40  0001 C CNN
 F 2 "" H 5650 4000 60  0000 C CNN
@@
 $EndComp
 $Comp
-L +3.3V #PWR503
+L +3.3V #PWR058
 U 1 1 54B2F47D
 P 6750 3300
-F 0 "#PWR503" H 6750 3390 20  0001 C CNN
+F 0 "#PWR058" H 6750 3390 20  0001 C CNN
 F 1 "+3.3V" H 6750 3390 30  0000 C CNN
 F 2 "" H 6750 3300 60  0000 C CNN
@@
 $EndComp
 $Comp
-L GNDPWR #PWR504
+L GNDPWR #PWR059
 U 1 1 54B2F483
 P 6750 3700
-F 0 "#PWR504" H 6750 3750 40  0001 C CNN
+F 0 "#PWR059" H 6750 3750 40  0001 C CNN
 F 1 "GNDPWR" H 6750 3620 40  0001 C CNN
 F 2 "" H 6750 3700 60  0000 C CNN
@@
 	5650 3500 5750 3500
 Wire Wire Line
-	5650 2900 5650 2950
-Wire Wire Line
-	5650 2950 5650 3500
+	5650 2900 5650 3500
 Wire Wire Line
 	5750 3700 5650 3700
@@
 	5750 3800 4800 3800
 Wire Wire Line
-	4800 3300 5500 3300
-Wire Wire Line
-	5500 3300 5750 3300
+	4800 3300 5750 3300
 Wire Wire Line
 	6750 3400 6750 3300

Commit message: initial layout
Parts:
- U501: footprint (none) -> kicadlib:AMPHENOL-114-00841-68
Changed lines of the file:
@@
 F 0 "U501" H 5950 4450 60  0000 L CNN
 F 1 "MICROSD-AMPHENOL-114-00841-68" H 5950 3450 60  0000 L CNN
-F 2 "" H 5950 3750 60  0001 C CNN
+F 2 "kicadlib:AMPHENOL-114-00841-68" H 5950 3750 60  0001 C CNN
 F 3 "" H 5950 3750 60  0000 C CNN
 	1    5950 3750
@@
 NoConn ~ 5750 3900
 $Comp
-L +3.3V #PWR056
+L +3.3V #PWR057
 U 1 1 54B2F466
 P 5650 2900
-F 0 "#PWR056" H 5650 2990 20  0001 C CNN
+F 0 "#PWR057" H 5650 2990 20  0001 C CNN
 F 1 "+3.3V" H 5650 2990 30  0000 C CNN
 F 2 "" H 5650 2900 60  0000 C CNN
@@
 $EndComp
 $Comp
-L GNDPWR #PWR057
+L GNDPWR #PWR058
 U 1 1 54B2F46C
 P 5650 4000
-F 0 "#PWR057" H 5650 4050 40  0001 C CNN
+F 0 "#PWR058" H 5650 4050 40  0001 C CNN
 F 1 "GNDPWR" H 5650 3920 40  0001 C CNN
 F 2 "" H 5650 4000 60  0000 C CNN
@@
 $EndComp
 $Comp
-L +3.3V #PWR058
+L +3.3V #PWR059
 U 1 1 54B2F47D
 P 6750 3300
-F 0 "#PWR058" H 6750 3390 20  0001 C CNN
+F 0 "#PWR059" H 6750 3390 20  0001 C CNN
 F 1 "+3.3V" H 6750 3390 30  0000 C CNN
 F 2 "" H 6750 3300 60  0000 C CNN
@@
 $EndComp
 $Comp
-L GNDPWR #PWR059
+L GNDPWR #PWR060
 U 1 1 54B2F483
 P 6750 3700
-F 0 "#PWR059" H 6750 3750 40  0001 C CNN
+F 0 "#PWR060" H 6750 3750 40  0001 C CNN
 F 1 "GNDPWR" H 6750 3620 40  0001 C CNN
 F 2 "" H 6750 3700 60  0000 C CNN

Commit message: v20150125
Parts:
- C501: inventoryId (none) -> 13
- R501: inventoryId (none) -> 299
- U501: inventoryId (none) -> 602
Changed lines of the file:
@@
 F 2 "kicadlib:AMPHENOL-114-00841-68" H 5950 3750 60  0001 C CNN
 F 3 "" H 5950 3750 60  0000 C CNN
+F 4 "602" H 5950 3750 60  0001 C CNN "inventoryId"
 	1    5950 3750
 	1    0    0    -1
@@
 F 2 "kicadlib:CAPC2012X100N" H 6750 3500 60  0001 C CNN
 F 3 "" H 6750 3500 60  0000 C CNN
+F 4 "13" H 6750 3500 60  0001 C CNN "inventoryId"
 	1    6750 3500
 	1    0    0    -1
@@
 F 2 "kicadlib:RESC2012X100N" H 5500 3100 60  0001 C CNN
 F 3 "" H 5500 3100 60  0000 C CNN
+F 4 "299" H 5500 3100 60  0001 C CNN "inventoryId"
 	1    5500 3100
 	-1   0    0    1
