File: hardware/stm32-wifi-door-bell-wifi.sch (KiCad schematic (older format))
At the start: 11 parts, among them P3 P03, U3 TICC3000, X3 ANT

Commit message: reannotate schematic
Parts:
- renumbered C13 to C401, C14 to C402, C15 to C403, C17 to C404, L2 to L401, L3 to L402, P3 to P401, R5 to R401, R6 to R402, U3 to U401, X3 to X401
Changed lines of the file:
@@
 $EndDescr
 $Comp
-L TICC3000 U3
+L TICC3000 U401
 U 1 1 54B2B952
 P 5400 3800
-F 0 "U3" H 4700 5350 60  0000 L CNN
+F 0 "U401" H 4700 5350 60  0000 L CNN
 F 1 "TICC3000" H 4700 2450 60  0000 L CNN
 F 2 "" H 6900 3800 60  0000 C CNN
@@
 $EndComp
 $Comp
-L GNDPWR #PWR52
+L GNDPWR #PWR404
 U 1 1 54B2B959
 P 4400 5100
-F 0 "#PWR52" H 4400 5150 40  0001 C CNN
+F 0 "#PWR404" H 4400 5150 40  0001 C CNN
 F 1 "GNDPWR" H 4400 5020 40  0001 C CNN
 F 2 "" H 4400 5100 60  0000 C CNN
@@
 	6400 3400 6300 3400
 $Comp
-L P03 P3
+L P03 P401
 U 1 1 54B2B995
 P 7100 3800
-F 0 "P3" H 7150 3855 60  0000 C CNN
+F 0 "P401" H 7150 3855 60  0000 C CNN
 F 1 "P03" H 7175 3345 60  0000 C CNN
 F 2 "" H 7100 3800 60  0000 C CNN
@@
 $EndComp
 $Comp
-L GNDPWR #PWR55
+L GNDPWR #PWR407
 U 1 1 54B2B99C
 P 6800 4200
-F 0 "#PWR55" H 6800 4250 40  0001 C CNN
+F 0 "#PWR407" H 6800 4250 40  0001 C CNN
 F 1 "GNDPWR" H 6800 4120 40  0001 C CNN
 F 2 "" H 6800 4200 60  0000 C CNN
@@
 CC3000RX
 $Comp
-L +3.3V #PWR51
+L +3.3V #PWR403
 U 1 1 54B2B9A4
 P 4400 2300
-F 0 "#PWR51" H 4400 2390 20  0001 C CNN
+F 0 "#PWR403" H 4400 2390 20  0001 C CNN
 F 1 "+3.3V" H 4400 2390 30  0000 C CNN
 F 2 "" H 4400 2300 60  0000 C CNN
@@
 Connection ~ 4400 2400
 $Comp
-L C C14
+L C C402
 U 1 1 54B2B9AE
 P 4000 2500
-F 0 "C14" H 4025 2550 30  0000 L CNN
+F 0 "C402" H 4025 2550 30  0000 L CNN
 F 1 "0.1uF" H 4025 2450 30  0000 L CNN
 F 2 "kicadlib:CAPC2012X100N" H 4000 2500 60  0001 C CNN
@@
 $EndComp
 $Comp
-L C C13
+L C C401
 U 1 1 54B2B9B5
 P 3800 2500
-F 0 "C13" H 3825 2550 30  0000 L CNN
+F 0 "C401" H 3825 2550 30  0000 L CNN
 F 1 "0.1uF" H 3825 2450 30  0000 L CNN
 F 2 "kicadlib:CAPC2012X100N" H 3800 2500 60  0001 C CNN
@@
 $EndComp
 $Comp
-L +3.3V #PWR49
+L +3.3V #PWR401
 U 1 1 54B2B9BC
 P 3800 2300
-F 0 "#PWR49" H 3800 2390 20  0001 C CNN
+F 0 "#PWR401" H 3800 2390 20  0001 C CNN
 F 1 "+3.3V" H 3800 2390 30  0000 C CNN
 F 2 "" H 3800 2300 60  0000 C CNN
@@
 $EndComp
 $Comp
-L GNDPWR #PWR50
+L GNDPWR #PWR402
 U 1 1 54B2B9C2
 P 3800 2700
-F 0 "#PWR50" H 3800 2750 40  0001 C CNN
+F 0 "#PWR402" H 3800 2750 40  0001 C CNN
 F 1 "GNDPWR" H 3800 2620 40  0001 C CNN
 F 2 "" H 3800 2700 60  0000 C CNN
@@
 	6400 4300 6300 4300
 $Comp
-L C C15
+L C C403
 U 1 1 54B2B9E7
 P 7450 2400
-F 0 "C15" H 7475 2450 30  0000 L CNN
+F 0 "C403" H 7475 2450 30  0000 L CNN
 F 1 "10pF" H 7475 2350 30  0000 L CNN
 F 2 "kicadlib:CAPC2012X100N" H 7450 2400 60  0001 C CNN
@@
 $EndComp
 $Comp
-L GNDPWR #PWR56
+L GNDPWR #PWR408
 U 1 1 54B2B9EE
 P 7600 2900
-F 0 "#PWR56" H 7600 2950 40  0001 C CNN
+F 0 "#PWR408" H 7600 2950 40  0001 C CNN
 F 1 "GNDPWR" H 7600 2820 40  0001 C CNN
 F 2 "" H 7600 2900 60  0000 C CNN
@@
 	6300 2400 7350 2400
 $Comp
-L C C17
+L C C404
 U 1 1 54B2B9F5
 P 7750 2400
-F 0 "C17" H 7775 2450 30  0000 L CNN
+F 0 "C404" H 7775 2450 30  0000 L CNN
 F 1 "2.2pF" H 7775 2350 30  0000 L CNN
 F 2 "kicadlib:CAPC2012X100N" H 7750 2400 60  0001 C CNN
@@
 	7600 2750 7600 2900
 $Comp
-L GNDPWR #PWR57
+L GNDPWR #PWR409
 U 1 1 54B2BA02
 P 7900 2900
-F 0 "#PWR57" H 7900 2950 40  0001 C CNN
+F 0 "#PWR409" H 7900 2950 40  0001 C CNN
 F 1 "GNDPWR" H 7900 2820 40  0001 C CNN
 F 2 "" H 7900 2900 60  0000 C CNN
@@
 	7900 2750 7900 2900
 $Comp
-L INDUCTOR L2
+L INDUCTOR L401
 U 1 1 54B2BA09
 P 7600 2600
-F 0 "L2" H 7600 2550 30  0000 C CNN
+F 0 "L401" H 7600 2550 30  0000 C CNN
 F 1 "2.2nH" H 7600 2650 30  0000 C CNN
 F 2 "" H 7600 2600 60  0000 C CNN
@@
 $EndComp
 $Comp
-L INDUCTOR L3
+L INDUCTOR L402
 U 1 1 54B2BA10
 P 7900 2600
-F 0 "L3" H 7900 2550 30  0000 C CNN
+F 0 "L402" H 7900 2550 30  0000 C CNN
 F 1 "DNP" H 7900 2650 30  0000 C CNN
 F 2 "" H 7900 2600 60  0000 C CNN
@@
 $EndComp
 $Comp
-L ANT X3
+L ANT X401
 U 1 1 54B2BA17
 P 7900 2150
-F 0 "X3" H 8000 2300 60  0000 L CNN
+F 0 "X401" H 8000 2300 60  0000 L CNN
 F 1 "ANT" H 8000 2200 60  0000 L CNN
 F 2 "" H 7900 2250 60  0000 C CNN
@@
 Connection ~ 7900 2400
 $Comp
-L R R6
+L R R402
 U 1 1 54B2BA1F
 P 6750 3450
-F 0 "R6" V 6695 3450 30  0000 C CNN
+F 0 "R402" V 6695 3450 30  0000 C CNN
 F 1 "10K" V 6650 3450 30  0000 C CNN
 F 2 "kicadlib:RESC2012X100N" H 6750 3450 60  0001 C CNN
@@
 $EndComp
 $Comp
-L R R5
+L R R401
 U 1 1 54B2BA26
 P 6750 2050
-F 0 "R5" V 6695 2050 30  0000 C CNN
+F 0 "R401" V 6695 2050 30  0000 C CNN
 F 1 "10K" V 6650 2050 30  0000 C CNN
 F 2 "kicadlib:RESC2012X100N" H 6750 2050 60  0001 C CNN
@@
 Connection ~ 6750 3200
 $Comp
-L +3.3V #PWR53
+L +3.3V #PWR405
 U 1 1 54B2BA30
 P 6750 1850
-F 0 "#PWR53" H 6750 1940 20  0001 C CNN
+F 0 "#PWR405" H 6750 1940 20  0001 C CNN
 F 1 "+3.3V" H 6750 1940 30  0000 C CNN
 F 2 "" H 6750 1850 60  0000 C CNN
@@
 	6750 1950 6750 1850
 $Comp
-L GNDPWR #PWR54
+L GNDPWR #PWR406
 U 1 1 54B2BA37
 P 6750 3650
-F 0 "#PWR54" H 6750 3700 40  0001 C CNN
+F 0 "#PWR406" H 6750 3700 40  0001 C CNN
 F 1 "GNDPWR" H 6750 3570 40  0001 C CNN
 F 2 "" H 6750 3650 60  0000 C CNN

Commit message: more schematics
Parts:
- P401: footprint (none) -> kicadlib:HDRV3W66P254_1X3_762X249X838P
Changed lines of the file:
@@
 F 0 "U401" H 4700 5350 60  0000 L CNN
 F 1 "TICC3000" H 4700 2450 60  0000 L CNN
-F 2 "" H 6900 3800 60  0000 C CNN
+F 2 "" H 6900 3800 60  0001 C CNN
 F 3 "" H 6900 3800 60  0000 C CNN
 	1    5400 3800
@@
 $EndComp
 $Comp
-L GNDPWR #PWR404
+L GNDPWR #PWR047
 U 1 1 54B2B959
 P 4400 5100
-F 0 "#PWR404" H 4400 5150 40  0001 C CNN
+F 0 "#PWR047" H 4400 5150 40  0001 C CNN
 F 1 "GNDPWR" H 4400 5020 40  0001 C CNN
 F 2 "" H 4400 5100 60  0000 C CNN
@@
 F 0 "P401" H 7150 3855 60  0000 C CNN
 F 1 "P03" H 7175 3345 60  0000 C CNN
-F 2 "" H 7100 3800 60  0000 C CNN
+F 2 "kicadlib:HDRV3W66P254_1X3_762X249X838P" H 7100 3800 60  0001 C CNN
 F 3 "" H 7100 3800 60  0000 C CNN
 	1    7100 3800
@@
 $EndComp
 $Comp
-L GNDPWR #PWR407
+L GNDPWR #PWR048
 U 1 1 54B2B99C
 P 6800 4200
-F 0 "#PWR407" H 6800 4250 40  0001 C CNN
+F 0 "#PWR048" H 6800 4250 40  0001 C CNN
 F 1 "GNDPWR" H 6800 4120 40  0001 C CNN
 F 2 "" H 6800 4200 60  0000 C CNN
@@
 CC3000RX
 $Comp
-L +3.3V #PWR403
+L +3.3V #PWR049
 U 1 1 54B2B9A4
 P 4400 2300
-F 0 "#PWR403" H 4400 2390 20  0001 C CNN
+F 0 "#PWR049" H 4400 2390 20  0001 C CNN
 F 1 "+3.3V" H 4400 2390 30  0000 C CNN
 F 2 "" H 4400 2300 60  0000 C CNN
@@
 $EndComp
 $Comp
-L +3.3V #PWR401
+L +3.3V #PWR050
 U 1 1 54B2B9BC
 P 3800 2300
-F 0 "#PWR401" H 3800 2390 20  0001 C CNN
+F 0 "#PWR050" H 3800 2390 20  0001 C CNN
 F 1 "+3.3V" H 3800 2390 30  0000 C CNN
 F 2 "" H 3800 2300 60  0000 C CNN
@@
 $EndComp
 $Comp
-L GNDPWR #PWR402
+L GNDPWR #PWR051
 U 1 1 54B2B9C2
 P 3800 2700
-F 0 "#PWR402" H 3800 2750 40  0001 C CNN
+F 0 "#PWR051" H 3800 2750 40  0001 C CNN
 F 1 "GNDPWR" H 3800 2620 40  0001 C CNN
 F 2 "" H 3800 2700 60  0000 C CNN
@@
 $EndComp
 $Comp
-L GNDPWR #PWR408
+L GNDPWR #PWR052
 U 1 1 54B2B9EE
 P 7600 2900
-F 0 "#PWR408" H 7600 2950 40  0001 C CNN
+F 0 "#PWR052" H 7600 2950 40  0001 C CNN
 F 1 "GNDPWR" H 7600 2820 40  0001 C CNN
 F 2 "" H 7600 2900 60  0000 C CNN
@@
 	7600 2750 7600 2900
 $Comp
-L GNDPWR #PWR409
+L GNDPWR #PWR053
 U 1 1 54B2BA02
 P 7900 2900
-F 0 "#PWR409" H 7900 2950 40  0001 C CNN
+F 0 "#PWR053" H 7900 2950 40  0001 C CNN
 F 1 "GNDPWR" H 7900 2820 40  0001 C CNN
 F 2 "" H 7900 2900 60  0000 C CNN
@@
 F 0 "L401" H 7600 2550 30  0000 C CNN
 F 1 "2.2nH" H 7600 2650 30  0000 C CNN
-F 2 "" H 7600 2600 60  0000 C CNN
+F 2 "" H 7600 2600 60  0001 C CNN
 F 3 "" H 7600 2600 60  0000 C CNN
 	1    7600 2600
@@
 F 0 "L402" H 7900 2550 30  0000 C CNN
 F 1 "DNP" H 7900 2650 30  0000 C CNN
-F 2 "" H 7900 2600 60  0000 C CNN
+F 2 "" H 7900 2600 60  0001 C CNN
 F 3 "" H 7900 2600 60  0000 C CNN
 	1    7900 2600
@@
 F 0 "X401" H 8000 2300 60  0000 L CNN
 F 1 "ANT" H 8000 2200 60  0000 L CNN
-F 2 "" H 7900 2250 60  0000 C CNN
+F 2 "" H 7900 2250 60  0001 C CNN
 F 3 "" H 7900 2250 60  0000 C CNN
 	1    7900 2150
@@
 Connection ~ 6750 3200
 $Comp
-L +3.3V #PWR405
+L +3.3V #PWR054
 U 1 1 54B2BA30
 P 6750 1850
-F 0 "#PWR405" H 6750 1940 20  0001 C CNN
+F 0 "#PWR054" H 6750 1940 20  0001 C CNN
 F 1 "+3.3V" H 6750 1940 30  0000 C CNN
 F 2 "" H 6750 1850 60  0000 C CNN
@@
 	6750 1950 6750 1850
 $Comp
-L GNDPWR #PWR406
+L GNDPWR #PWR055
 U 1 1 54B2BA37
 P 6750 3650
-F 0 "#PWR406" H 6750 3700 40  0001 C CNN
+F 0 "#PWR055" H 6750 3700 40  0001 C CNN
 F 1 "GNDPWR" H 6750 3570 40  0001 C CNN
 F 2 "" H 6750 3650 60  0000 C CNN

Commit message: initial layout
Parts:
- L401, L402: footprint (none) -> kicadlib:INDC1005X60N; MfgPartNumber (none) -> L-07C2N2SV6T
- U401: footprint (none) -> kicadlib:TI-CC3000
- X401: value ANT -> 2500AT44M0400E; footprint (none) -> kicadlib:JT-2500AT44M0400E
Changed lines of the file:
@@
 F 0 "U401" H 4700 5350 60  0000 L CNN
 F 1 "TICC3000" H 4700 2450 60  0000 L CNN
-F 2 "" H 6900 3800 60  0001 C CNN
+F 2 "kicadlib:TI-CC3000" H 6900 3800 60  0001 C CNN
 F 3 "" H 6900 3800 60  0000 C CNN
 	1    5400 3800
@@
 $EndComp
 $Comp
-L GNDPWR #PWR047
+L GNDPWR #PWR048
 U 1 1 54B2B959
 P 4400 5100
-F 0 "#PWR047" H 4400 5150 40  0001 C CNN
+F 0 "#PWR048" H 4400 5150 40  0001 C CNN
 F 1 "GNDPWR" H 4400 5020 40  0001 C CNN
 F 2 "" H 4400 5100 60  0000 C CNN
@@
 $EndComp
 $Comp
-L GNDPWR #PWR048
+L GNDPWR #PWR049
 U 1 1 54B2B99C
 P 6800 4200
-F 0 "#PWR048" H 6800 4250 40  0001 C CNN
+F 0 "#PWR049" H 6800 4250 40  0001 C CNN
 F 1 "GNDPWR" H 6800 4120 40  0001 C CNN
 F 2 "" H 6800 4200 60  0000 C CNN
@@
 CC3000RX
 $Comp
-L +3.3V #PWR049
+L +3.3V #PWR050
 U 1 1 54B2B9A4
 P 4400 2300
-F 0 "#PWR049" H 4400 2390 20  0001 C CNN
+F 0 "#PWR050" H 4400 2390 20  0001 C CNN
 F 1 "+3.3V" H 4400 2390 30  0000 C CNN
 F 2 "" H 4400 2300 60  0000 C CNN
@@
 $EndComp
 $Comp
-L +3.3V #PWR050
+L +3.3V #PWR051
 U 1 1 54B2B9BC
 P 3800 2300
-F 0 "#PWR050" H 3800 2390 20  0001 C CNN
+F 0 "#PWR051" H 3800 2390 20  0001 C CNN
 F 1 "+3.3V" H 3800 2390 30  0000 C CNN
 F 2 "" H 3800 2300 60  0000 C CNN
@@
 $EndComp
 $Comp
-L GNDPWR #PWR051
+L GNDPWR #PWR052
 U 1 1 54B2B9C2
 P 3800 2700
-F 0 "#PWR051" H 3800 2750 40  0001 C CNN
+F 0 "#PWR052" H 3800 2750 40  0001 C CNN
 F 1 "GNDPWR" H 3800 2620 40  0001 C CNN
 F 2 "" H 3800 2700 60  0000 C CNN
@@
 $EndComp
 $Comp
-L GNDPWR #PWR052
+L GNDPWR #PWR053
 U 1 1 54B2B9EE
 P 7600 2900
-F 0 "#PWR052" H 7600 2950 40  0001 C CNN
+F 0 "#PWR053" H 7600 2950 40  0001 C CNN
 F 1 "GNDPWR" H 7600 2820 40  0001 C CNN
 F 2 "" H 7600 2900 60  0000 C CNN
@@
 	7600 2750 7600 2900
 $Comp
-L GNDPWR #PWR053
+L GNDPWR #PWR054
 U 1 1 54B2BA02
 P 7900 2900
-F 0 "#PWR053" H 7900 2950 40  0001 C CNN
+F 0 "#PWR054" H 7900 2950 40  0001 C CNN
 F 1 "GNDPWR" H 7900 2820 40  0001 C CNN
 F 2 "" H 7900 2900 60  0000 C CNN
@@
 F 0 "L401" H 7600 2550 30  0000 C CNN
 F 1 "2.2nH" H 7600 2650 30  0000 C CNN
-F 2 "" H 7600 2600 60  0001 C CNN
+F 2 "kicadlib:INDC1005X60N" H 7600 2600 60  0001 C CNN
 F 3 "" H 7600 2600 60  0000 C CNN
+F 4 "L-07C2N2SV6T" H 7600 2600 60  0001 C CNN "MfgPartNumber"
 	1    7600 2600
 	0    1    1    0
@@
 F 0 "L402" H 7900 2550 30  0000 C CNN
 F 1 "DNP" H 7900 2650 30  0000 C CNN
-F 2 "" H 7900 2600 60  0001 C CNN
+F 2 "kicadlib:INDC1005X60N" H 7900 2600 60  0001 C CNN
 F 3 "" H 7900 2600 60  0000 C CNN
+F 4 "L-07C2N2SV6T" H 7900 2600 60  0001 C CNN "MfgPartNumber"
 	1    7900 2600
 	0    1    1    0
@@
 P 7900 2150
 F 0 "X401" H 8000 2300 60  0000 L CNN
-F 1 "ANT" H 8000 2200 60  0000 L CNN
-F 2 "" H 7900 2250 60  0001 C CNN
+F 1 "2500AT44M0400E" H 8000 2200 60  0000 L CNN
+F 2 "kicadlib:JT-2500AT44M0400E" H 7900 2250 60  0001 C CNN
 F 3 "" H 7900 2250 60  0000 C CNN
 	1    7900 2150
@@
 Connection ~ 6750 3200
 $Comp
-L +3.3V #PWR054
+L +3.3V #PWR055
 U 1 1 54B2BA30
 P 6750 1850
-F 0 "#PWR054" H 6750 1940 20  0001 C CNN
+F 0 "#PWR055" H 6750 1940 20  0001 C CNN
 F 1 "+3.3V" H 6750 1940 30  0000 C CNN
 F 2 "" H 6750 1850 60  0000 C CNN
@@
 	6750 1950 6750 1850
 $Comp
-L GNDPWR #PWR055
+L GNDPWR #PWR056
 U 1 1 54B2BA37
 P 6750 3650
-F 0 "#PWR055" H 6750 3700 40  0001 C CNN
+F 0 "#PWR056" H 6750 3700 40  0001 C CNN
 F 1 "GNDPWR" H 6750 3570 40  0001 C CNN
 F 2 "" H 6750 3650 60  0000 C CNN

Commit message: clean up pcb
Connections:
- net ANT-NET-0: now reaches C403.1, U401.35 (RFANT)
- net ANT-NET-1: now reaches C403.2, C404.1, L401.1
- net ANT-NET-2: now reaches C404.2, L402.1, X401.0
Changed lines of the file:
@@
 $EndComp
 $Comp
-L GNDPWR #PWR048
+L GNDPWR #PWR051
 U 1 1 54B2B959
 P 4400 5100
-F 0 "#PWR048" H 4400 5150 40  0001 C CNN
+F 0 "#PWR051" H 4400 5150 40  0001 C CNN
 F 1 "GNDPWR" H 4400 5020 40  0001 C CNN
 F 2 "" H 4400 5100 60  0000 C CNN
@@
 $EndComp
 $Comp
-L GNDPWR #PWR049
+L GNDPWR #PWR052
 U 1 1 54B2B99C
 P 6800 4200
-F 0 "#PWR049" H 6800 4250 40  0001 C CNN
+F 0 "#PWR052" H 6800 4250 40  0001 C CNN
 F 1 "GNDPWR" H 6800 4120 40  0001 C CNN
 F 2 "" H 6800 4200 60  0000 C CNN
@@
 CC3000RX
 $Comp
-L +3.3V #PWR050
+L +3.3V #PWR053
 U 1 1 54B2B9A4
 P 4400 2300
-F 0 "#PWR050" H 4400 2390 20  0001 C CNN
+F 0 "#PWR053" H 4400 2390 20  0001 C CNN
 F 1 "+3.3V" H 4400 2390 30  0000 C CNN
 F 2 "" H 4400 2300 60  0000 C CNN
@@
 $EndComp
 $Comp
-L +3.3V #PWR051
+L +3.3V #PWR054
 U 1 1 54B2B9BC
 P 3800 2300
-F 0 "#PWR051" H 3800 2390 20  0001 C CNN
+F 0 "#PWR054" H 3800 2390 20  0001 C CNN
 F 1 "+3.3V" H 3800 2390 30  0000 C CNN
 F 2 "" H 3800 2300 60  0000 C CNN
@@
 $EndComp
 $Comp
-L GNDPWR #PWR052
+L GNDPWR #PWR055
 U 1 1 54B2B9C2
 P 3800 2700
-F 0 "#PWR052" H 3800 2750 40  0001 C CNN
+F 0 "#PWR055" H 3800 2750 40  0001 C CNN
 F 1 "GNDPWR" H 3800 2620 40  0001 C CNN
 F 2 "" H 3800 2700 60  0000 C CNN
@@
 $EndComp
 $Comp
-L GNDPWR #PWR053
+L GNDPWR #PWR056
 U 1 1 54B2B9EE
 P 7600 2900
-F 0 "#PWR053" H 7600 2950 40  0001 C CNN
+F 0 "#PWR056" H 7600 2950 40  0001 C CNN
 F 1 "GNDPWR" H 7600 2820 40  0001 C CNN
 F 2 "" H 7600 2900 60  0000 C CNN
@@
 	7600 2750 7600 2900
 $Comp
-L GNDPWR #PWR054
+L GNDPWR #PWR057
 U 1 1 54B2BA02
 P 7900 2900
-F 0 "#PWR054" H 7900 2950 40  0001 C CNN
+F 0 "#PWR057" H 7900 2950 40  0001 C CNN
 F 1 "GNDPWR" H 7900 2820 40  0001 C CNN
 F 2 "" H 7900 2900 60  0000 C CNN
@@
 Connection ~ 6750 3200
 $Comp
-L +3.3V #PWR055
+L +3.3V #PWR058
 U 1 1 54B2BA30
 P 6750 1850
-F 0 "#PWR055" H 6750 1940 20  0001 C CNN
+F 0 "#PWR058" H 6750 1940 20  0001 C CNN
 F 1 "+3.3V" H 6750 1940 30  0000 C CNN
 F 2 "" H 6750 1850 60  0000 C CNN
@@
 	6750 1950 6750 1850
 $Comp
-L GNDPWR #PWR056
+L GNDPWR #PWR059
 U 1 1 54B2BA37
 P 6750 3650
-F 0 "#PWR056" H 6750 3700 40  0001 C CNN
+F 0 "#PWR059" H 6750 3700 40  0001 C CNN
 F 1 "GNDPWR" H 6750 3570 40  0001 C CNN
 F 2 "" H 6750 3650 60  0000 C CNN
@@
 Wire Wire Line
 	6300 3100 6900 3100
+Text Label 6900 2400 0    20   ~ 0
+ANT-NET-0
+Text Label 7600 2400 1    20   ~ 0
+ANT-NET-1
+Text Label 7900 2350 1    20   ~ 0
+ANT-NET-2
 $EndSCHEMATC

Commit message: v20150125
Parts:
- C401, C402: inventoryId (none) -> 10
- C403: inventoryId (none) -> 606
- C404: inventoryId (none) -> 607
- L401: inventoryId (none) -> 599
- L402, P401: inventoryId (none) -> NA
- R401, R402: inventoryId (none) -> 299
- U401: inventoryId (none) -> 598
- X401: inventoryId (none) -> 597
Changed lines of the file:
@@
 F 2 "kicadlib:TI-CC3000" H 6900 3800 60  0001 C CNN
 F 3 "" H 6900 3800 60  0000 C CNN
+F 4 "598" H 5400 3800 60  0001 C CNN "inventoryId"
 	1    5400 3800
 	1    0    0    -1
@@
 F 2 "kicadlib:HDRV3W66P254_1X3_762X249X838P" H 7100 3800 60  0001 C CNN
 F 3 "" H 7100 3800 60  0000 C CNN
+F 4 "NA" H 7100 3800 60  0001 C CNN "inventoryId"
 	1    7100 3800
 	1    0    0    -1
@@
 F 2 "kicadlib:CAPC2012X100N" H 4000 2500 60  0001 C CNN
 F 3 "" H 4000 2500 60  0000 C CNN
+F 4 "10" H 4000 2500 60  0001 C CNN "inventoryId"
 	1    4000 2500
 	1    0    0    -1
@@
 F 2 "kicadlib:CAPC2012X100N" H 3800 2500 60  0001 C CNN
 F 3 "" H 3800 2500 60  0000 C CNN
+F 4 "10" H 3800 2500 60  0001 C CNN "inventoryId"
 	1    3800 2500
 	1    0    0    -1
@@
 F 2 "kicadlib:CAPC2012X100N" H 7450 2400 60  0001 C CNN
 F 3 "" H 7450 2400 60  0000 C CNN
+F 4 "606" H 7450 2400 60  0001 C CNN "inventoryId"
 	1    7450 2400
 	0    -1   -1   0
@@
 F 2 "kicadlib:CAPC2012X100N" H 7750 2400 60  0001 C CNN
 F 3 "" H 7750 2400 60  0000 C CNN
+F 4 "607" H 7750 2400 60  0001 C CNN "inventoryId"
 	1    7750 2400
 	0    -1   -1   0
@@
 F 3 "" H 7600 2600 60  0000 C CNN
 F 4 "L-07C2N2SV6T" H 7600 2600 60  0001 C CNN "MfgPartNumber"
+F 5 "599" H 7600 2600 60  0001 C CNN "inventoryId"
 	1    7600 2600
 	0    1    1    0
@@
 F 3 "" H 7900 2600 60  0000 C CNN
 F 4 "L-07C2N2SV6T" H 7900 2600 60  0001 C CNN "MfgPartNumber"
+F 5 "NA" H 7900 2600 60  0001 C CNN "inventoryId"
 	1    7900 2600
 	0    1    1    0
@@
 F 2 "kicadlib:JT-2500AT44M0400E" H 7900 2250 60  0001 C CNN
 F 3 "" H 7900 2250 60  0000 C CNN
+F 4 "597" H 7900 2150 60  0001 C CNN "inventoryId"
 	1    7900 2150
 	1    0    0    -1
@@
 F 2 "kicadlib:RESC2012X100N" H 6750 3450 60  0001 C CNN
 F 3 "" H 6750 3450 60  0000 C CNN
+F 4 "299" H 6750 3450 60  0001 C CNN "inventoryId"
 	1    6750 3450
 	-1   0    0    1
@@
 F 2 "kicadlib:RESC2012X100N" H 6750 2050 60  0001 C CNN
 F 3 "" H 6750 2050 60  0000 C CNN
+F 4 "299" H 6750 2050 60  0001 C CNN "inventoryId"
 	1    6750 2050
 	-1   0    0    1
