File: hardware/stm32-wifi-door-bell-audio.sch (KiCad schematic (older format))
At the start: 15 parts

Commit message: reannotate schematic
Parts:
- added R604, R607: 0R, symbol R
- gave numbers to parts that had none: 15
Connections:
- wire segments 34 -> 36
Changed lines of the file:
@@
 AUDIOIN
 $Comp
-L P02 P?
+L P02 P601
 U 1 1 54B32862
 P 7250 2900
-F 0 "P?" H 7300 2950 60  0000 C CNN
+F 0 "P601" H 7300 2950 60  0000 C CNN
 F 1 "SPEAKER" H 7250 2550 60  0000 L CNN
 F 2 "" H 7250 2900 60  0000 C CNN
@@
 $EndComp
 $Comp
-L GNDPWR #PWR?
+L GNDPWR #PWR610
 U 1 1 54B32E66
 P 6950 3200
-F 0 "#PWR?" H 6950 3250 40  0001 C CNN
+F 0 "#PWR610" H 6950 3250 40  0001 C CNN
 F 1 "GNDPWR" H 6950 3120 40  0001 C CNN
 F 2 "" H 6950 3200 60  0000 C CNN
@@
 	6950 3100 6950 3200
 $Comp
-L LM1875 U?
+L LM1875 U601
 U 1 1 54B33194
 P 5200 3000
-F 0 "U?" H 5400 2850 60  0000 L CNN
+F 0 "U601" H 5400 2850 60  0000 L CNN
 F 1 "LM1875" H 5400 2750 60  0000 L CNN
 F 2 "" H 5200 3000 60  0000 C CNN
@@
 	5600 3000 6550 3000
 $Comp
-L R R?
+L R R608
 U 1 1 54B33211
 P 6300 3200
-F 0 "R?" V 6245 3200 30  0000 C CNN
+F 0 "R608" V 6245 3200 30  0000 C CNN
 F 1 "1R" V 6355 3200 30  0000 C CNN
 F 2 "" H 6300 3200 60  0000 C CNN
@@
 $EndComp
 $Comp
-L C C?
+L C C606
 U 1 1 54B33269
 P 6300 3500
-F 0 "C?" H 6325 3550 30  0000 L CNN
+F 0 "C606" H 6325 3550 30  0000 L CNN
 F 1 "0.22uF" H 6325 3450 30  0000 L CNN
 F 2 "" H 6300 3500 60  0000 C CNN
@@
 	6300 3300 6300 3400
 $Comp
-L GNDPWR #PWR?
+L GNDPWR #PWR609
 U 1 1 54B332B0
 P 6300 3700
-F 0 "#PWR?" H 6300 3750 40  0001 C CNN
+F 0 "#PWR609" H 6300 3750 40  0001 C CNN
 F 1 "GNDPWR" H 6300 3620 40  0001 C CNN
 F 2 "" H 6300 3700 60  0000 C CNN
@@
 	4900 3100 4800 3100
 $Comp
-L C C?
+L C C601
 U 1 1 54B3342C
 P 3800 2900
-F 0 "C?" H 3825 2950 30  0000 L CNN
+F 0 "C601" H 3825 2950 30  0000 L CNN
 F 1 "1uF" H 3825 2850 30  0000 L CNN
 F 2 "" H 3800 2900 60  0000 C CNN
@@
 $EndComp
 $Comp
-L R R?
+L R R601
 U 1 1 54B334DB
 P 3600 3100
-F 0 "R?" V 3545 3100 30  0000 C CNN
+F 0 "R601" V 3545 3100 30  0000 C CNN
 F 1 "1M" V 3655 3100 30  0000 C CNN
 F 2 "" H 3600 3100 60  0000 C CNN
@@
 	3900 2900 4900 2900
 $Comp
-L CP C?
+L CP C603
 U 1 1 54B335C3
-P 4600 3850
-F 0 "C?" H 4625 3900 30  0000 L CNN
-F 1 "10uF" H 4625 3800 30  0000 L CNN
-F 2 "" H 4600 3850 60  0000 C CNN
-F 3 "" H 4600 3850 60  0000 C CNN
-	1    4600 3850
-	1    0    0    -1
-$EndComp
-$Comp
-L GNDPWR #PWR?
+P 4600 4100
+F 0 "C603" H 4625 4150 30  0000 L CNN
+F 1 "10uF" H 4625 4050 30  0000 L CNN
+F 2 "" H 4600 4100 60  0000 C CNN
+F 3 "" H 4600 4100 60  0000 C CNN
+	1    4600 4100
+	1    0    0    -1
+$EndComp
+$Comp
+L GNDPWR #PWR604
 U 1 1 54B3361E
-P 4600 4050
-F 0 "#PWR?" H 4600 4100 40  0001 C CNN
-F 1 "GNDPWR" H 4600 3970 40  0001 C CNN
-F 2 "" H 4600 4050 60  0000 C CNN
-F 3 "" H 4600 4050 60  0000 C CNN
-	1    4600 4050
-	1    0    0    -1
-$EndComp
-Wire Wire Line
-	4600 3950 4600 4050
-$Comp
-L GNDPWR #PWR?
+P 4600 4300
+F 0 "#PWR604" H 4600 4350 40  0001 C CNN
+F 1 "GNDPWR" H 4600 4220 40  0001 C CNN
+F 2 "" H 4600 4300 60  0000 C CNN
+F 3 "" H 4600 4300 60  0000 C CNN
+	1    4600 4300
+	1    0    0    -1
+$EndComp
+Wire Wire Line
+	4600 4200 4600 4300
+$Comp
+L GNDPWR #PWR601
 U 1 1 54B33698
 P 3600 3300
-F 0 "#PWR?" H 3600 3350 40  0001 C CNN
+F 0 "#PWR601" H 3600 3350 40  0001 C CNN
 F 1 "GNDPWR" H 3600 3220 40  0001 C CNN
 F 2 "" H 3600 3300 60  0000 C CNN
@@
 	3600 3200 3600 3300
 $Comp
-L GNDPWR #PWR?
+L GNDPWR #PWR606
 U 1 1 54B336F2
 P 5200 3400
-F 0 "#PWR?" H 5200 3450 40  0001 C CNN
+F 0 "#PWR606" H 5200 3450 40  0001 C CNN
 F 1 "GNDPWR" H 5200 3320 40  0001 C CNN
 F 2 "" H 5200 3400 60  0000 C CNN
@@
 	5200 3300 5200 3400
 $Comp
-L CP C?
+L CP C604
 U 1 1 54B33763
 P 6000 2200
-F 0 "C?" H 6025 2250 30  0000 L CNN
+F 0 "C604" H 6025 2250 30  0000 L CNN
 F 1 "100uF" H 6025 2150 30  0000 L CNN
 F 2 "" H 6000 2200 60  0000 C CNN
@@
 $EndComp
 $Comp
-L C C?
+L C C605
 U 1 1 54B33820
 P 6300 2200
-F 0 "C?" H 6325 2250 30  0000 L CNN
+F 0 "C605" H 6325 2250 30  0000 L CNN
 F 1 "0.1uF" H 6325 2150 30  0000 L CNN
 F 2 "" H 6300 2200 60  0000 C CNN
@@
 $EndComp
 $Comp
-L GNDPWR #PWR?
+L GNDPWR #PWR608
 U 1 1 54B338CA
 P 6300 2500
-F 0 "#PWR?" H 6300 2550 40  0001 C CNN
+F 0 "#PWR608" H 6300 2550 40  0001 C CNN
 F 1 "GNDPWR" H 6300 2420 40  0001 C CNN
 F 2 "" H 6300 2500 60  0000 C CNN
@@
 Connection ~ 6300 2400
 $Comp
-L Vcc #PWR?
+L Vcc #PWR607
 U 1 1 54B3392A
 P 6000 1900
-F 0 "#PWR?" H 6000 1990 20  0001 C CNN
+F 0 "#PWR607" H 6000 1990 20  0001 C CNN
 F 1 "Vcc" H 6000 1990 30  0000 C CNN
 F 2 "" H 6000 1900 60  0000 C CNN
@@
 $EndComp
 $Comp
-L Vcc #PWR?
+L Vcc #PWR605
 U 1 1 54B33948
 P 5200 2200
-F 0 "#PWR?" H 5200 2290 20  0001 C CNN
+F 0 "#PWR605" H 5200 2290 20  0001 C CNN
 F 1 "Vcc" H 5200 2290 30  0000 C CNN
 F 2 "" H 5200 2200 60  0000 C CNN
@@
 	6000 2400 6000 2300
 $Comp
-L CP C?
+L CP C607
 U 1 1 54B33CDC
 P 6650 3000
-F 0 "C?" H 6675 3050 30  0000 L CNN
+F 0 "C607" H 6675 3050 30  0000 L CNN
 F 1 "2200uF" H 6675 2950 30  0000 L CNN
 F 2 "" H 6650 3000 60  0000 C CNN
@@
 	7050 3000 6750 3000
 $Comp
-L R R?
+L R R603
 U 1 1 54B33EFD
 P 4600 2500
-F 0 "R?" V 4545 2500 30  0000 C CNN
+F 0 "R603" V 4545 2500 30  0000 C CNN
 F 1 "22K" V 4655 2500 30  0000 C CNN
 F 2 "" H 4600 2500 60  0000 C CNN
@@
 $EndComp
 $Comp
-L R R?
+L R R605
 U 1 1 54B33FA7
 P 4800 2350
-F 0 "R?" V 4745 2350 30  0000 C CNN
+F 0 "R605" V 4745 2350 30  0000 C CNN
 F 1 "22K" V 4855 2350 30  0000 C CNN
 F 2 "" H 4800 2350 60  0000 C CNN
@@
 Connection ~ 4600 2900
 $Comp
-L R R?
+L R R602
 U 1 1 54B340FA
 P 4150 2500
-F 0 "R?" V 4095 2500 30  0000 C CNN
+F 0 "R602" V 4095 2500 30  0000 C CNN
 F 1 "22K" V 4205 2500 30  0000 C CNN
 F 2 "" H 4150 2500 60  0000 C CNN
@@
 $EndComp
 $Comp
-L CP C?
+L CP C602
 U 1 1 54B341EF
 P 4350 2500
-F 0 "C?" H 4375 2550 30  0000 L CNN
+F 0 "C602" H 4375 2550 30  0000 L CNN
 F 1 "10uF" H 4375 2450 30  0000 L CNN
 F 2 "" H 4350 2500 60  0000 C CNN
@@
 Connection ~ 4350 2350
 $Comp
-L GNDPWR #PWR?
+L GNDPWR #PWR602
 U 1 1 54B34309
 P 4150 2700
-F 0 "#PWR?" H 4150 2750 40  0001 C CNN
+F 0 "#PWR602" H 4150 2750 40  0001 C CNN
 F 1 "GNDPWR" H 4150 2620 40  0001 C CNN
 F 2 "" H 4150 2700 60  0000 C CNN
@@
 	4350 2600 4350 2700
 $Comp
-L GNDPWR #PWR?
+L GNDPWR #PWR603
 U 1 1 54B343B9
 P 4350 2700
-F 0 "#PWR?" H 4350 2750 40  0001 C CNN
+F 0 "#PWR603" H 4350 2750 40  0001 C CNN
 F 1 "GNDPWR" H 4350 2620 40  0001 C CNN
 F 2 "" H 4350 2700 60  0000 C CNN
@@
 $EndComp
 $Comp
-L POT R?
+L POT R606
 U 1 1 54B2C9F5
 P 4800 3550
-F 0 "R?" V 4745 3550 30  0000 C CNN
+F 0 "R606" V 4745 3550 30  0000 C CNN
 F 1 "100K" V 4865 3530 30  0000 R CNN
 F 2 "" H 4800 3550 60  0000 C CNN
@@
 $EndComp
 Wire Wire Line
-	4900 3550 6000 3550
-Wire Wire Line
 	4800 3100 4800 3450
 Wire Wire Line
 	4700 3550 4600 3550
-Wire Wire Line
-	4600 3550 4600 3750
+$Comp
+L R R607
+U 1 1 54B3134D
+P 5100 3550
+F 0 "R607" V 5045 3550 30  0000 C CNN
+F 1 "0R" V 5155 3550 30  0000 C CNN
+F 2 "" H 5100 3550 60  0000 C CNN
+F 3 "" H 5100 3550 60  0000 C CNN
+	1    5100 3550
+	0    1    1    0
+$EndComp
+$Comp
+L R R604
+U 1 1 54B31434
+P 4600 3750
+F 0 "R604" V 4545 3750 30  0000 C CNN
+F 1 "0R" V 4655 3750 30  0000 C CNN
+F 2 "" H 4600 3750 60  0000 C CNN
+F 3 "" H 4600 3750 60  0000 C CNN
+	1    4600 3750
+	-1   0    0    1
+$EndComp
+Wire Wire Line
+	4900 3550 5000 3550
+Wire Wire Line
+	5200 3550 6000 3550
+Wire Wire Line
+	4600 3550 4600 3650
+Wire Wire Line
+	4600 3850 4600 4000
 $EndSCHEMATC

Commit message: more schematics
Parts:
- C601, C605, C606: footprint (none) -> kicadlib:CAPC2012X100N
- C602, C603: footprint (none) -> kicadlib:CAPCP2012X100N
- P601: footprint (none) -> kicadlib:OST-OSTTC022162; MfgPartNumber (none) -> OSTTC022162
- R601, R602, R603, R604, R605, R607, R608: footprint (none) -> kicadlib:RESC2012X100N
- R606: footprint (none) -> kicadlib:COPAL-CT6EP
Changed lines of the file:
@@
 F 0 "P601" H 7300 2950 60  0000 C CNN
 F 1 "SPEAKER" H 7250 2550 60  0000 L CNN
-F 2 "" H 7250 2900 60  0000 C CNN
+F 2 "kicadlib:OST-OSTTC022162" H 7250 2900 60  0001 C CNN
 F 3 "" H 7250 2900 60  0000 C CNN
+F 4 "OSTTC022162" H 7250 2900 60  0001 C CNN "MfgPartNumber"
 	1    7250 2900
 	1    0    0    -1
 $EndComp
 $Comp
-L GNDPWR #PWR610
+L GNDPWR #PWR060
 U 1 1 54B32E66
 P 6950 3200
-F 0 "#PWR610" H 6950 3250 40  0001 C CNN
+F 0 "#PWR060" H 6950 3250 40  0001 C CNN
 F 1 "GNDPWR" H 6950 3120 40  0001 C CNN
 F 2 "" H 6950 3200 60  0000 C CNN
@@
 F 0 "U601" H 5400 2850 60  0000 L CNN
 F 1 "LM1875" H 5400 2750 60  0000 L CNN
-F 2 "" H 5200 3000 60  0000 C CNN
+F 2 "" H 5200 3000 60  0001 C CNN
 F 3 "" H 5200 3000 60  0000 C CNN
 	1    5200 3000
@@
 F 0 "R608" V 6245 3200 30  0000 C CNN
 F 1 "1R" V 6355 3200 30  0000 C CNN
-F 2 "" H 6300 3200 60  0000 C CNN
+F 2 "kicadlib:RESC2012X100N" H 6300 3200 60  0001 C CNN
 F 3 "" H 6300 3200 60  0000 C CNN
 	1    6300 3200
@@
 F 0 "C606" H 6325 3550 30  0000 L CNN
 F 1 "0.22uF" H 6325 3450 30  0000 L CNN
-F 2 "" H 6300 3500 60  0000 C CNN
+F 2 "kicadlib:CAPC2012X100N" H 6300 3500 60  0001 C CNN
 F 3 "" H 6300 3500 60  0000 C CNN
 	1    6300 3500
@@
 	6300 3300 6300 3400
 $Comp
-L GNDPWR #PWR609
+L GNDPWR #PWR061
 U 1 1 54B332B0
 P 6300 3700
-F 0 "#PWR609" H 6300 3750 40  0001 C CNN
+F 0 "#PWR061" H 6300 3750 40  0001 C CNN
 F 1 "GNDPWR" H 6300 3620 40  0001 C CNN
 F 2 "" H 6300 3700 60  0000 C CNN
@@
 F 0 "C601" H 3825 2950 30  0000 L CNN
 F 1 "1uF" H 3825 2850 30  0000 L CNN
-F 2 "" H 3800 2900 60  0000 C CNN
+F 2 "kicadlib:CAPC2012X100N" H 3800 2900 60  0001 C CNN
 F 3 "" H 3800 2900 60  0000 C CNN
 	1    3800 2900
@@
 F 0 "R601" V 3545 3100 30  0000 C CNN
 F 1 "1M" V 3655 3100 30  0000 C CNN
-F 2 "" H 3600 3100 60  0000 C CNN
+F 2 "kicadlib:RESC2012X100N" H 3600 3100 60  0001 C CNN
 F 3 "" H 3600 3100 60  0000 C CNN
 	1    3600 3100
@@
 F 0 "C603" H 4625 4150 30  0000 L CNN
 F 1 "10uF" H 4625 4050 30  0000 L CNN
-F 2 "" H 4600 4100 60  0000 C CNN
+F 2 "kicadlib:CAPCP2012X100N" H 4600 4100 60  0001 C CNN
 F 3 "" H 4600 4100 60  0000 C CNN
 	1    4600 4100
@@
 $EndComp
 $Comp
-L GNDPWR #PWR604
+L GNDPWR #PWR062
 U 1 1 54B3361E
 P 4600 4300
-F 0 "#PWR604" H 4600 4350 40  0001 C CNN
+F 0 "#PWR062" H 4600 4350 40  0001 C CNN
 F 1 "GNDPWR" H 4600 4220 40  0001 C CNN
 F 2 "" H 4600 4300 60  0000 C CNN
@@
 	4600 4200 4600 4300
 $Comp
-L GNDPWR #PWR601
+L GNDPWR #PWR063
 U 1 1 54B33698
 P 3600 3300
-F 0 "#PWR601" H 3600 3350 40  0001 C CNN
+F 0 "#PWR063" H 3600 3350 40  0001 C CNN
 F 1 "GNDPWR" H 3600 3220 40  0001 C CNN
 F 2 "" H 3600 3300 60  0000 C CNN
@@
 	3600 3200 3600 3300
 $Comp
-L GNDPWR #PWR606
+L GNDPWR #PWR064
 U 1 1 54B336F2
 P 5200 3400
-F 0 "#PWR606" H 5200 3450 40  0001 C CNN
+F 0 "#PWR064" H 5200 3450 40  0001 C CNN
 F 1 "GNDPWR" H 5200 3320 40  0001 C CNN
 F 2 "" H 5200 3400 60  0000 C CNN
@@
 F 0 "C604" H 6025 2250 30  0000 L CNN
 F 1 "100uF" H 6025 2150 30  0000 L CNN
-F 2 "" H 6000 2200 60  0000 C CNN
+F 2 "" H 6000 2200 60  0001 C CNN
 F 3 "" H 6000 2200 60  0000 C CNN
 	1    6000 2200
@@
 F 0 "C605" H 6325 2250 30  0000 L CNN
 F 1 "0.1uF" H 6325 2150 30  0000 L CNN
-F 2 "" H 6300 2200 60  0000 C CNN
+F 2 "kicadlib:CAPC2012X100N" H 6300 2200 60  0001 C CNN
 F 3 "" H 6300 2200 60  0000 C CNN
 	1    6300 2200
@@
 $EndComp
 $Comp
-L GNDPWR #PWR608
+L GNDPWR #PWR065
 U 1 1 54B338CA
 P 6300 2500
-F 0 "#PWR608" H 6300 2550 40  0001 C CNN
+F 0 "#PWR065" H 6300 2550 40  0001 C CNN
 F 1 "GNDPWR" H 6300 2420 40  0001 C CNN
 F 2 "" H 6300 2500 60  0000 C CNN
@@
 Connection ~ 6300 2400
 $Comp
-L Vcc #PWR607
+L Vcc #PWR066
 U 1 1 54B3392A
 P 6000 1900
-F 0 "#PWR607" H 6000 1990 20  0001 C CNN
+F 0 "#PWR066" H 6000 1990 20  0001 C CNN
 F 1 "Vcc" H 6000 1990 30  0000 C CNN
 F 2 "" H 6000 1900 60  0000 C CNN
@@
 $EndComp
 $Comp
-L Vcc #PWR605
+L Vcc #PWR067
 U 1 1 54B33948
 P 5200 2200
-F 0 "#PWR605" H 5200 2290 20  0001 C CNN
+F 0 "#PWR067" H 5200 2290 20  0001 C CNN
 F 1 "Vcc" H 5200 2290 30  0000 C CNN
 F 2 "" H 5200 2200 60  0000 C CNN
@@
 F 0 "C607" H 6675 3050 30  0000 L CNN
 F 1 "2200uF" H 6675 2950 30  0000 L CNN
-F 2 "" H 6650 3000 60  0000 C CNN
+F 2 "" H 6650 3000 60  0001 C CNN
 F 3 "" H 6650 3000 60  0000 C CNN
 	1    6650 3000
@@
 F 0 "R603" V 4545 2500 30  0000 C CNN
 F 1 "22K" V 4655 2500 30  0000 C CNN
-F 2 "" H 4600 2500 60  0000 C CNN
+F 2 "kicadlib:RESC2012X100N" H 4600 2500 60  0001 C CNN
 F 3 "" H 4600 2500 60  0000 C CNN
 	1    4600 2500
@@
 F 0 "R605" V 4745 2350 30  0000 C CNN
 F 1 "22K" V 4855 2350 30  0000 C CNN
-F 2 "" H 4800 2350 60  0000 C CNN
+F 2 "kicadlib:RESC2012X100N" H 4800 2350 60  0001 C CNN
 F 3 "" H 4800 2350 60  0000 C CNN
 	1    4800 2350
@@
 F 0 "R602" V 4095 2500 30  0000 C CNN
 F 1 "22K" V 4205 2500 30  0000 C CNN
-F 2 "" H 4150 2500 60  0000 C CNN
+F 2 "kicadlib:RESC2012X100N" H 4150 2500 60  0001 C CNN
 F 3 "" H 4150 2500 60  0000 C CNN
 	1    4150 2500
@@
 F 0 "C602" H 4375 2550 30  0000 L CNN
 F 1 "10uF" H 4375 2450 30  0000 L CNN
-F 2 "" H 4350 2500 60  0000 C CNN
+F 2 "kicadlib:CAPCP2012X100N" H 4350 2500 60  0001 C CNN
 F 3 "" H 4350 2500 60  0000 C CNN
 	1    4350 2500
@@
 Connection ~ 4350 2350
 $Comp
-L GNDPWR #PWR602
+L GNDPWR #PWR068
 U 1 1 54B34309
 P 4150 2700
-F 0 "#PWR602" H 4150 2750 40  0001 C CNN
+F 0 "#PWR068" H 4150 2750 40  0001 C CNN
 F 1 "GNDPWR" H 4150 2620 40  0001 C CNN
 F 2 "" H 4150 2700 60  0000 C CNN
@@
 	4350 2600 4350 2700
 $Comp
-L GNDPWR #PWR603
+L GNDPWR #PWR069
 U 1 1 54B343B9
 P 4350 2700
-F 0 "#PWR603" H 4350 2750 40  0001 C CNN
+F 0 "#PWR069" H 4350 2750 40  0001 C CNN
 F 1 "GNDPWR" H 4350 2620 40  0001 C CNN
 F 2 "" H 4350 2700 60  0000 C CNN
@@
 F 0 "R606" V 4745 3550 30  0000 C CNN
 F 1 "100K" V 4865 3530 30  0000 R CNN
-F 2 "" H 4800 3550 60  0000 C CNN
+F 2 "kicadlib:COPAL-CT6EP" H 4800 3550 60  0001 C CNN
 F 3 "" H 4800 3550 60  0000 C CNN
 	1    4800 3550
@@
 F 0 "R607" V 5045 3550 30  0000 C CNN
 F 1 "0R" V 5155 3550 30  0000 C CNN
-F 2 "" H 5100 3550 60  0000 C CNN
+F 2 "kicadlib:RESC2012X100N" H 5100 3550 60  0001 C CNN
 F 3 "" H 5100 3550 60  0000 C CNN
 	1    5100 3550
@@
 F 0 "R604" V 4545 3750 30  0000 C CNN
 F 1 "0R" V 4655 3750 30  0000 C CNN
-F 2 "" H 4600 3750 60  0000 C CNN
+F 2 "kicadlib:RESC2012X100N" H 4600 3750 60  0001 C CNN
 F 3 "" H 4600 3750 60  0000 C CNN
 	1    4600 3750

Commit message: initial layout
Parts:
- C604: footprint (none) -> kicadlib:CAPAE660X790N
- C607: value 2200uF -> 2200uF >16V; footprint (none) -> kicadlib:CAPPRD750W80D1600H2500P
- U601: footprint (none) -> kicadlib:TO170P470X1028X2117-5P
Changed lines of the file:
@@
 $EndComp
 $Comp
-L GNDPWR #PWR060
+L GNDPWR #PWR061
 U 1 1 54B32E66
 P 6950 3200
-F 0 "#PWR060" H 6950 3250 40  0001 C CNN
+F 0 "#PWR061" H 6950 3250 40  0001 C CNN
 F 1 "GNDPWR" H 6950 3120 40  0001 C CNN
 F 2 "" H 6950 3200 60  0000 C CNN
@@
 F 0 "U601" H 5400 2850 60  0000 L CNN
 F 1 "LM1875" H 5400 2750 60  0000 L CNN
-F 2 "" H 5200 3000 60  0001 C CNN
+F 2 "kicadlib:TO170P470X1028X2117-5P" H 5200 3000 60  0001 C CNN
 F 3 "" H 5200 3000 60  0000 C CNN
 	1    5200 3000
@@
 	6300 3300 6300 3400
 $Comp
-L GNDPWR #PWR061
+L GNDPWR #PWR062
 U 1 1 54B332B0
 P 6300 3700
-F 0 "#PWR061" H 6300 3750 40  0001 C CNN
+F 0 "#PWR062" H 6300 3750 40  0001 C CNN
 F 1 "GNDPWR" H 6300 3620 40  0001 C CNN
 F 2 "" H 6300 3700 60  0000 C CNN
@@
 $EndComp
 $Comp
-L GNDPWR #PWR062
+L GNDPWR #PWR063
 U 1 1 54B3361E
 P 4600 4300
-F 0 "#PWR062" H 4600 4350 40  0001 C CNN
+F 0 "#PWR063" H 4600 4350 40  0001 C CNN
 F 1 "GNDPWR" H 4600 4220 40  0001 C CNN
 F 2 "" H 4600 4300 60  0000 C CNN
@@
 	4600 4200 4600 4300
 $Comp
-L GNDPWR #PWR063
+L GNDPWR #PWR064
 U 1 1 54B33698
 P 3600 3300
-F 0 "#PWR063" H 3600 3350 40  0001 C CNN
+F 0 "#PWR064" H 3600 3350 40  0001 C CNN
 F 1 "GNDPWR" H 3600 3220 40  0001 C CNN
 F 2 "" H 3600 3300 60  0000 C CNN
@@
 	3600 3200 3600 3300
 $Comp
-L GNDPWR #PWR064
+L GNDPWR #PWR065
 U 1 1 54B336F2
 P 5200 3400
-F 0 "#PWR064" H 5200 3450 40  0001 C CNN
+F 0 "#PWR065" H 5200 3450 40  0001 C CNN
 F 1 "GNDPWR" H 5200 3320 40  0001 C CNN
 F 2 "" H 5200 3400 60  0000 C CNN
@@
 F 0 "C604" H 6025 2250 30  0000 L CNN
 F 1 "100uF" H 6025 2150 30  0000 L CNN
-F 2 "" H 6000 2200 60  0001 C CNN
+F 2 "kicadlib:CAPAE660X790N" H 6000 2200 60  0001 C CNN
 F 3 "" H 6000 2200 60  0000 C CNN
 	1    6000 2200
@@
 $EndComp
 $Comp
-L GNDPWR #PWR065
+L GNDPWR #PWR066
 U 1 1 54B338CA
 P 6300 2500
-F 0 "#PWR065" H 6300 2550 40  0001 C CNN
+F 0 "#PWR066" H 6300 2550 40  0001 C CNN
 F 1 "GNDPWR" H 6300 2420 40  0001 C CNN
 F 2 "" H 6300 2500 60  0000 C CNN
@@
 Connection ~ 6300 2400
 $Comp
-L Vcc #PWR066
+L Vcc #PWR067
 U 1 1 54B3392A
 P 6000 1900
-F 0 "#PWR066" H 6000 1990 20  0001 C CNN
+F 0 "#PWR067" H 6000 1990 20  0001 C CNN
 F 1 "Vcc" H 6000 1990 30  0000 C CNN
 F 2 "" H 6000 1900 60  0000 C CNN
@@
 $EndComp
 $Comp
-L Vcc #PWR067
+L Vcc #PWR068
 U 1 1 54B33948
 P 5200 2200
-F 0 "#PWR067" H 5200 2290 20  0001 C CNN
+F 0 "#PWR068" H 5200 2290 20  0001 C CNN
 F 1 "Vcc" H 5200 2290 30  0000 C CNN
 F 2 "" H 5200 2200 60  0000 C CNN
@@
 P 6650 3000
 F 0 "C607" H 6675 3050 30  0000 L CNN
-F 1 "2200uF" H 6675 2950 30  0000 L CNN
-F 2 "" H 6650 3000 60  0001 C CNN
+F 1 "2200uF >16V" H 6675 2950 30  0000 L CNN
+F 2 "kicadlib:CAPPRD750W80D1600H2500P" H 6650 3000 60  0001 C CNN
 F 3 "" H 6650 3000 60  0000 C CNN
 	1    6650 3000
@@
 Connection ~ 4350 2350
 $Comp
-L GNDPWR #PWR068
+L GNDPWR #PWR069
 U 1 1 54B34309
 P 4150 2700
-F 0 "#PWR068" H 4150 2750 40  0001 C CNN
+F 0 "#PWR069" H 4150 2750 40  0001 C CNN
 F 1 "GNDPWR" H 4150 2620 40  0001 C CNN
 F 2 "" H 4150 2700 60  0000 C CNN
@@
 	4350 2600 4350 2700
 $Comp
-L GNDPWR #PWR069
+L GNDPWR #PWR070
 U 1 1 54B343B9
 P 4350 2700
-F 0 "#PWR069" H 4350 2750 40  0001 C CNN
+F 0 "#PWR070" H 4350 2750 40  0001 C CNN
 F 1 "GNDPWR" H 4350 2620 40  0001 C CNN
 F 2 "" H 4350 2700 60  0000 C CNN

Commit message: clean up pcb
Parts:
- P601: footprint kicadlib:OST-OSTTC022162 -> kicadlib:OST-OSTTA024163
Changed lines of the file:
@@
 F 0 "P601" H 7300 2950 60  0000 C CNN
 F 1 "SPEAKER" H 7250 2550 60  0000 L CNN
-F 2 "kicadlib:OST-OSTTC022162" H 7250 2900 60  0001 C CNN
+F 2 "kicadlib:OST-OSTTA024163" H 7250 2900 60  0001 C CNN
 F 3 "" H 7250 2900 60  0000 C CNN
 F 4 "OSTTC022162" H 7250 2900 60  0001 C CNN "MfgPartNumber"
@@
 $EndComp
 $Comp
-L GNDPWR #PWR061
+L GNDPWR #PWR064
 U 1 1 54B32E66
 P 6950 3200
-F 0 "#PWR061" H 6950 3250 40  0001 C CNN
+F 0 "#PWR064" H 6950 3250 40  0001 C CNN
 F 1 "GNDPWR" H 6950 3120 40  0001 C CNN
 F 2 "" H 6950 3200 60  0000 C CNN
@@
 	6300 3300 6300 3400
 $Comp
-L GNDPWR #PWR062
+L GNDPWR #PWR065
 U 1 1 54B332B0
 P 6300 3700
-F 0 "#PWR062" H 6300 3750 40  0001 C CNN
+F 0 "#PWR065" H 6300 3750 40  0001 C CNN
 F 1 "GNDPWR" H 6300 3620 40  0001 C CNN
 F 2 "" H 6300 3700 60  0000 C CNN
@@
 $EndComp
 $Comp
-L GNDPWR #PWR063
+L GNDPWR #PWR066
 U 1 1 54B3361E
 P 4600 4300
-F 0 "#PWR063" H 4600 4350 40  0001 C CNN
+F 0 "#PWR066" H 4600 4350 40  0001 C CNN
 F 1 "GNDPWR" H 4600 4220 40  0001 C CNN
 F 2 "" H 4600 4300 60  0000 C CNN
@@
 	4600 4200 4600 4300
 $Comp
-L GNDPWR #PWR064
+L GNDPWR #PWR067
 U 1 1 54B33698
 P 3600 3300
-F 0 "#PWR064" H 3600 3350 40  0001 C CNN
+F 0 "#PWR067" H 3600 3350 40  0001 C CNN
 F 1 "GNDPWR" H 3600 3220 40  0001 C CNN
 F 2 "" H 3600 3300 60  0000 C CNN
@@
 	3600 3200 3600 3300
 $Comp
-L GNDPWR #PWR065
+L GNDPWR #PWR068
 U 1 1 54B336F2
 P 5200 3400
-F 0 "#PWR065" H 5200 3450 40  0001 C CNN
+F 0 "#PWR068" H 5200 3450 40  0001 C CNN
 F 1 "GNDPWR" H 5200 3320 40  0001 C CNN
 F 2 "" H 5200 3400 60  0000 C CNN
@@
 $EndComp
 $Comp
-L GNDPWR #PWR066
+L GNDPWR #PWR069
 U 1 1 54B338CA
 P 6300 2500
-F 0 "#PWR066" H 6300 2550 40  0001 C CNN
+F 0 "#PWR069" H 6300 2550 40  0001 C CNN
 F 1 "GNDPWR" H 6300 2420 40  0001 C CNN
 F 2 "" H 6300 2500 60  0000 C CNN
@@
 Connection ~ 6300 2400
 $Comp
-L Vcc #PWR067
+L Vcc #PWR070
 U 1 1 54B3392A
 P 6000 1900
-F 0 "#PWR067" H 6000 1990 20  0001 C CNN
+F 0 "#PWR070" H 6000 1990 20  0001 C CNN
 F 1 "Vcc" H 6000 1990 30  0000 C CNN
 F 2 "" H 6000 1900 60  0000 C CNN
@@
 $EndComp
 $Comp
-L Vcc #PWR068
+L Vcc #PWR071
 U 1 1 54B33948
 P 5200 2200
-F 0 "#PWR068" H 5200 2290 20  0001 C CNN
+F 0 "#PWR071" H 5200 2290 20  0001 C CNN
 F 1 "Vcc" H 5200 2290 30  0000 C CNN
 F 2 "" H 5200 2200 60  0000 C CNN
@@
 Connection ~ 4350 2350
 $Comp
-L GNDPWR #PWR069
+L GNDPWR #PWR072
 U 1 1 54B34309
 P 4150 2700
-F 0 "#PWR069" H 4150 2750 40  0001 C CNN
+F 0 "#PWR072" H 4150 2750 40  0001 C CNN
 F 1 "GNDPWR" H 4150 2620 40  0001 C CNN
 F 2 "" H 4150 2700 60  0000 C CNN
@@
 	4350 2600 4350 2700
 $Comp
-L GNDPWR #PWR070
+L GNDPWR #PWR073
 U 1 1 54B343B9
 P 4350 2700
-F 0 "#PWR070" H 4350 2750 40  0001 C CNN
+F 0 "#PWR073" H 4350 2750 40  0001 C CNN
 F 1 "GNDPWR" H 4350 2620 40  0001 C CNN
 F 2 "" H 4350 2700 60  0000 C CNN
