File: hardware/stm32-wifi-door-bell-audio.sch (KiCad schematic (older format))
At the start: 17 parts, among them P601 SPEAKER, U601 LM1875

Commit message: v20150125
Parts:
- C601: inventoryId (none) -> 13
- C602, C603: inventoryId (none) -> 389
- C604: inventoryId (none) -> 464
- C605: inventoryId (none) -> 10
- C606: inventoryId (none) -> 605
- C607: inventoryId (none) -> 601
- P601: inventoryId (none) -> 603
- R601: inventoryId (none) -> 530
- R602, R603, R605: inventoryId (none) -> 612
- R604, R607: inventoryId (none) -> 430
- R606: inventoryId (none) -> 409
- R608: inventoryId (none) -> 611
- U601: inventoryId (none) -> 596
Changed lines of the file:
@@
 F 3 "" H 7250 2900 60  0000 C CNN
 F 4 "OSTTC022162" H 7250 2900 60  0001 C CNN "MfgPartNumber"
+F 5 "603" H 7250 2900 60  0001 C CNN "inventoryId"
 	1    7250 2900
 	1    0    0    -1
@@
 F 2 "kicadlib:TO170P470X1028X2117-5P" H 5200 3000 60  0001 C CNN
 F 3 "" H 5200 3000 60  0000 C CNN
+F 4 "596" H 5200 3000 60  0001 C CNN "inventoryId"
 	1    5200 3000
 	1    0    0    -1
@@
 F 2 "kicadlib:RESC2012X100N" H 6300 3200 60  0001 C CNN
 F 3 "" H 6300 3200 60  0000 C CNN
+F 4 "611" H 6300 3200 60  0001 C CNN "inventoryId"
 	1    6300 3200
 	1    0    0    -1
@@
 F 2 "kicadlib:CAPC2012X100N" H 6300 3500 60  0001 C CNN
 F 3 "" H 6300 3500 60  0000 C CNN
+F 4 "605" H 6300 3500 60  0001 C CNN "inventoryId"
 	1    6300 3500
 	1    0    0    -1
@@
 F 2 "kicadlib:CAPC2012X100N" H 3800 2900 60  0001 C CNN
 F 3 "" H 3800 2900 60  0000 C CNN
+F 4 "13" H 3800 2900 60  0001 C CNN "inventoryId"
 	1    3800 2900
 	0    1    1    0
@@
 F 2 "kicadlib:RESC2012X100N" H 3600 3100 60  0001 C CNN
 F 3 "" H 3600 3100 60  0000 C CNN
+F 4 "530" H 3600 3100 60  0001 C CNN "inventoryId"
 	1    3600 3100
 	1    0    0    -1
@@
 F 2 "kicadlib:CAPCP2012X100N" H 4600 4100 60  0001 C CNN
 F 3 "" H 4600 4100 60  0000 C CNN
+F 4 "389" H 4600 4100 60  0001 C CNN "inventoryId"
 	1    4600 4100
 	1    0    0    -1
@@
 F 2 "kicadlib:CAPAE660X790N" H 6000 2200 60  0001 C CNN
 F 3 "" H 6000 2200 60  0000 C CNN
+F 4 "464" H 6000 2200 60  0001 C CNN "inventoryId"
 	1    6000 2200
 	1    0    0    -1
@@
 F 2 "kicadlib:CAPC2012X100N" H 6300 2200 60  0001 C CNN
 F 3 "" H 6300 2200 60  0000 C CNN
+F 4 "10" H 6300 2200 60  0001 C CNN "inventoryId"
 	1    6300 2200
 	1    0    0    -1
@@
 F 2 "kicadlib:CAPPRD750W80D1600H2500P" H 6650 3000 60  0001 C CNN
 F 3 "" H 6650 3000 60  0000 C CNN
+F 4 "601" H 6650 3000 60  0001 C CNN "inventoryId"
 	1    6650 3000
 	0    -1   -1   0
@@
 F 2 "kicadlib:RESC2012X100N" H 4600 2500 60  0001 C CNN
 F 3 "" H 4600 2500 60  0000 C CNN
+F 4 "612" H 4600 2500 60  0001 C CNN "inventoryId"
 	1    4600 2500
 	1    0    0    -1
@@
 F 2 "kicadlib:RESC2012X100N" H 4800 2350 60  0001 C CNN
 F 3 "" H 4800 2350 60  0000 C CNN
+F 4 "612" H 4800 2350 60  0001 C CNN "inventoryId"
 	1    4800 2350
 	0    1    1    0
@@
 F 2 "kicadlib:RESC2012X100N" H 4150 2500 60  0001 C CNN
 F 3 "" H 4150 2500 60  0000 C CNN
+F 4 "612" H 4150 2500 60  0001 C CNN "inventoryId"
 	1    4150 2500
 	-1   0    0    1
@@
 F 2 "kicadlib:CAPCP2012X100N" H 4350 2500 60  0001 C CNN
 F 3 "" H 4350 2500 60  0000 C CNN
+F 4 "389" H 4350 2500 60  0001 C CNN "inventoryId"
 	1    4350 2500
 	1    0    0    -1
@@
 F 2 "kicadlib:COPAL-CT6EP" H 4800 3550 60  0001 C CNN
 F 3 "" H 4800 3550 60  0000 C CNN
+F 4 "409" H 4800 3550 60  0001 C CNN "inventoryId"
 	1    4800 3550
 	0    -1   -1   0
@@
 F 2 "kicadlib:RESC2012X100N" H 5100 3550 60  0001 C CNN
 F 3 "" H 5100 3550 60  0000 C CNN
+F 4 "430" H 5100 3550 60  0001 C CNN "inventoryId"
 	1    5100 3550
 	0    1    1    0
@@
 F 2 "kicadlib:RESC2012X100N" H 4600 3750 60  0001 C CNN
 F 3 "" H 4600 3750 60  0000 C CNN
+F 4 "430" H 4600 3750 60  0001 C CNN "inventoryId"
 	1    4600 3750
 	-1   0    0    1

Commit message: add speaker
Parts:
- added SPK1: Speaker, symbol MECH
Changed lines of the file:
@@
 Wire Wire Line
 	4600 3850 4600 4000
+$Comp
+L MECH SPK1
+U 1 1 54C63429
+P 6150 4300
+F 0 "SPK1" H 6200 4300 60  0000 C CNN
+F 1 "Speaker" H 6350 4300 60  0000 L CNN
+F 2 "" H 6150 4300 60  0000 C CNN
+F 3 "" H 6150 4300 60  0000 C CNN
+F 4 "614" H 6150 4300 60  0001 C CNN "inventoryId"
+	1    6150 4300
+	1    0    0    -1
+$EndComp
 $EndSCHEMATC
